File: hardware/ProstheticHandV2/untitled.kicad_sch (KiCad schematic)
At the start: 0 parts

Commit message: Update work on schematic
Other:
- note removed: "TODO - 3 potentiometers (one big, two trim pots) - 2 buttons Next sheet - 3 servo motors, current sensing for each and MOSFET to control the power/current they get - MOSFETs controlled by op-amps, where uC gives them using PWM signal and sets the max current"
Changed lines of the file:
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@@
 (kicad_sch (version 20230121) (generator eeschema)
   (paper "A4")
-  (text "TODO\n - 3 potentiometers (one big, two trim pots)\n - 2 buttons\n\nNext sheet\n - 3 servo motors, current sensing for each and \n   MOSFET to control the power/current they get\n - MOSFETs controlled by op-amps, where uC gives \n   them using PWM signal and sets the max current"
-    (at 38.1 104.14 0)
-    (effects (font (size 5 5)) (justify left bottom))
-  )
 )
