File: hardware/ProstheticHandV2/ProstheticHandV2.kicad_pcb (KiCad board)
At the start: 2 copper layers, 130 x 70 mm, 93 parts, among them J1 BATT_CONNECTOR, J2 EMG_SENSOR_01, J3 EMG_SENSOR_02, J4 CONN_SERVO_01, J6 CONN_SERVO_02, J7 CONN_SERVO_03, SW1 DIP_SWITCH, SW2 BUTTON_01, SW3 BUTTON_02, U1 LM7805_TO220

Commit message: Finalize PCB design for china
Parts:
- added TP3: TP_GND, TestPoint:TestPoint_Pad_D2.5mm, F.Cu at (120.0, 109.0)
- H1, H2, H3, H4: value MountingHole -> MountingHole_Pad; footprint MountingHole:MountingHole_3.2mm_M3 -> MountingHole:MountingHole_3.2mm_M3_Pad
- J1, J2, J3: footprint Connector_JST:JST_XA_B02B-XASK-1-A_1x02_P2.50mm_Vertical -> Connector_JST:JST_XA_B02B-XASK-1_1x02_P2.50mm_Vertical
- moved R1 120.0 mm to (222.0, 101.0), turned to -90 degrees
- moved R3 109.7 mm to (226.0, 108.6), turned to 90 degrees
- moved TP23 103.6 mm to (152.0, 108.0)
- moved C14 102.6 mm to (200.0, 89.0)
- moved TP25 102.5 mm to (140.0, 108.0)
- moved TP27 100.1 mm to (173.0, 115.0)
- moved C12 99.8 mm to (200.0, 82.0)
- moved C13 97.0 mm to (200.0, 75.0)
- moved C8 96.0 mm to (157.0, 69.0)
- moved C11 95.9 mm to (157.0, 64.0)
- moved TP29 95.3 mm to (180.0, 115.0)
- moved R10 94.7 mm to (142.2, 59.0)
- moved TP24 93.8 mm to (180.0, 109.0)
- moved R15 92.8 mm to (142.2, 54.0)
- moved TP26 92.4 mm to (180.0, 103.0)
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- renumbered C3 to C1, C9 to C10, C10 to C11, C14 to C12, C12 to C13, C15 to C14, C4 to C3, C1 to C4, C11 to C8, C8 to C9, D6 to D2, D4 to D3, D5 to D4, D2 to D5, D3 to D6, J6 to J4, J4 to J5, J7 to J6, R13 to R10, R10 to R11, R16 to R12, R17 to R13, R11 to R14, R14 to R15, R12 to R16, R15 to R17, R25 to R19, R9 to R2, R26 to R20, R23 to R22, R24 to R23, R19 to R24, R28 to R25, R29 to R26, R2 to R3, R5 to R4, R6 to R5, R7 to R6, R8 to R7, R3 to R8, R4 to R9, TP9 to TP10, TP17 to TP11, TP10 to TP12, TP15 to TP14, TP18 to TP15, TP11 to TP16, TP19 to TP17, TP12 to TP18, TP14 to TP19, TP16 to TP20, TP24 to TP21, TP20 to TP22, TP25 to TP23, TP29 to TP24, TP22 to TP25, TP28 to TP26, TP26 to TP27, TP27 to TP28, TP30 to TP29, TP5 to TP4, TP7 to TP5, TP8 to TP7, TP3 to TP8, TP4 to TP9
Connections:
- A1 pad 10: EMG_SENSOR_01 -> EMG_SENSOR_02
- A1 pad 11: EMG_SENSOR_02 -> EMG_SENSOR_01
- A1 pad 40: BUTTON_01 -> BUTTON_02
- A1 pad 41: BUTTON_02 -> BUTTON_01
Routing:
- net +BATT: track 0.00 -> 198.6 mm
- net +3V3: track 0.00 -> 150.0 mm, vias 0 -> 3
- net +5V: track 0.00 -> 149.2 mm, vias 0 -> 1
- net EMG_SENSOR_01: track 0.00 -> 114.0 mm, vias 0 -> 2
- net EMG_SENSOR_02: track 0.00 -> 109.2 mm, vias 0 -> 2
- net Net-(R16-Pad1): track 0.00 -> 75.9 mm, vias 0 -> 2
- net SERVO_CONTROL_03: track 0.00 -> 71.6 mm
- net SERVO_CONTROL_01: track 0.00 -> 69.8 mm
- net SERVO_CONTROL_02: track 0.00 -> 69.2 mm
- net Net-(J5-Pin_1): track 0.00 -> 66.1 mm, vias 0 -> 2
- net Net-(R14-Pad1): track 0.00 -> 52.2 mm, vias 0 -> 2
- net Net-(J4-Pin_1): track 0.00 -> 51.2 mm, vias 0 -> 2
- net Net-(R11-Pad1): track 0.00 -> 48.3 mm, vias 0 -> 2
- net Net-(J6-Pin_1): track 0.00 -> 44.6 mm, vias 0 -> 1
- net Net-(R15-Pad2): track 0.00 -> 40.0 mm
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- added copper zone on B.Cu, net GND
- added copper zone on F.Cu, net GND
Other:
- board text added: "+ -"
- board text added: "0 1 2 3"
- board text added: "1"
- board text added: "2"
- board text added: "3"
- board text added: "3v3"
- board text added: "5W 0.1Ω"
- board text added: "BATTERY"
- board text added: "BOOTSTRAP DIP SW"
- board text added: "BTN_01"
- board text added: "BTN_02"
- board text added: "DEBUG LED"
- board text added: "DEBUG_01"
- board text added: "DEBUG_02"
- board text added: "EMG_01"
- board text added: "EMG_02"
- board text added: "ESP32S3"
- board text added: "GND"
- board text added: "LM7805"
- board text added: "OFF - ON"
- board text added: "POT OUTPUT"
- board text added: "POT RAW"
- board text added: "PWR"
- board text added: "SERVO_01"
- board text added: "SERVO_02"
- board text added: "SERVO_03"
- board text added: "SIG VCC GND"
- board text added: "SIGN GND"
- board text added: "SRV_CTRL"
- board text added: "SRV_CURR"
