File: hardware/OpenHand/Control.kicad_sch (KiCad schematic)
At the start: 61 parts, among them U10 DRV8833PWP, U11 DRV8833PWP, U12 DRV8833PWP, U9 DRV8833PWP

Commit message: Update schm and pcb
Parts:
- renumbered R61 to R56, R62 to R57, R55 to R58, R56 to R59, R63 to R61, R57 to R62, R58 to R63, R59 to R64, TP30 to TP45, TP31 to TP46, TP32 to TP47, TP33 to TP48, TP34 to TP49, TP35 to TP50, TP36 to TP51, TP37 to TP52, TP38 to TP53, TP39 to TP54, TP40 to TP55, TP41 to TP56, TP42 to TP57, TP43 to TP58, TP44 to TP59, TP45 to TP60, TP46 to TP61, TP47 to TP62, TP48 to TP63, TP49 to TP64, TP50 to TP65, TP51 to TP66, TP52 to TP67, TP53 to TP68, TP54 to TP69, TP55 to TP70, TP56 to TP71, U9 to U10, U10 to U11, U11 to U12, U12 to U13

Commit message: Update schm and pcb
Parts:
- TP57: renamed from TP45; footprint (none) -> TestPoint:TestPoint_Pad_D1.0mm
- TP58: renamed from TP46; footprint (none) -> TestPoint:TestPoint_Pad_D1.0mm
- TP59: renamed from TP47; footprint (none) -> TestPoint:TestPoint_Pad_D1.0mm
- TP60: renamed from TP48; footprint (none) -> TestPoint:TestPoint_Pad_D1.0mm
- TP61: renamed from TP49; footprint (none) -> TestPoint:TestPoint_Pad_D1.0mm
- TP62: renamed from TP50; footprint (none) -> TestPoint:TestPoint_Pad_D1.0mm
- TP63: renamed from TP51; footprint (none) -> TestPoint:TestPoint_Pad_D1.0mm
- TP64: renamed from TP52; footprint (none) -> TestPoint:TestPoint_Pad_D1.0mm
- TP65: renamed from TP53; footprint (none) -> TestPoint:TestPoint_Pad_D1.0mm
- TP66: renamed from TP54; footprint (none) -> TestPoint:TestPoint_Pad_D1.0mm
- TP67: renamed from TP55; footprint (none) -> TestPoint:TestPoint_Pad_D1.0mm
- TP68: renamed from TP56; footprint (none) -> TestPoint:TestPoint_Pad_D1.0mm
- TP69: renamed from TP57; footprint (none) -> TestPoint:TestPoint_Pad_D1.0mm
- TP70: renamed from TP58; footprint (none) -> TestPoint:TestPoint_Pad_D1.0mm
- TP71: renamed from TP59; footprint (none) -> TestPoint:TestPoint_Pad_D1.0mm
- TP72: renamed from TP60; footprint (none) -> TestPoint:TestPoint_Pad_D1.0mm
- TP73: renamed from TP61; footprint (none) -> TestPoint:TestPoint_Pad_D1.0mm
- TP74: renamed from TP62; footprint (none) -> TestPoint:TestPoint_Pad_D1.0mm
- TP75: renamed from TP63; footprint (none) -> TestPoint:TestPoint_Pad_D1.0mm
- TP76: renamed from TP64; footprint (none) -> TestPoint:TestPoint_Pad_D1.0mm
- TP77: renamed from TP65; footprint (none) -> TestPoint:TestPoint_Pad_D1.0mm
- TP78: renamed from TP66; footprint (none) -> TestPoint:TestPoint_Pad_D1.0mm
- TP79: renamed from TP67; footprint (none) -> TestPoint:TestPoint_Pad_D1.0mm
- TP80: renamed from TP68; footprint (none) -> TestPoint:TestPoint_Pad_D1.0mm
- TP81: renamed from TP69; footprint (none) -> TestPoint:TestPoint_Pad_D1.0mm
- TP82: renamed from TP70; footprint (none) -> TestPoint:TestPoint_Pad_D1.0mm
- TP83: renamed from TP71; footprint (none) -> TestPoint:TestPoint_Pad_D1.0mm

Commit message: update schm and pcb again
Parts:
- renumbered TP57 to TP53, TP58 to TP54, TP59 to TP55, TP60 to TP56, TP61 to TP57, TP62 to TP58, TP63 to TP59, TP64 to TP60, TP65 to TP61, TP66 to TP62, TP67 to TP63, TP68 to TP64, TP69 to TP65, TP70 to TP66, TP71 to TP67, TP72 to TP68, TP73 to TP69, TP74 to TP70, TP75 to TP71, TP76 to TP72, TP77 to TP73, TP78 to TP74, TP79 to TP75, TP80 to TP76, TP81 to TP77, TP82 to TP78, TP83 to TP79
