File: hardware/OpenHand/Sensors.kicad_sch (KiCad schematic)
At the start: 9 parts, among them U3 INA333xxDGK, U4 OPA333xxDBV, U5 OPA333xxDBV, U6 ADS1115IDGS

Commit message: Minor updates to schm
Parts:
- removed U3: INA333xxDGK, Package_SO:VSSOP-8_3.0x3.0mm_P0.65mm, symbol Amplifier_Instrumentation:INA333xxDGK
- removed U4, U5: OPA333xxDBV, Package_TO_SOT_SMD:SOT-23-5, symbol Amplifier_Operational:OPA333xxDBV
- renumbered R8 to R12, R9 to R13, R10 to R14, R11 to R15, R12 to R16, U6 to U3
Changed lines of the file:
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@@
   (symbol (lib_id "Device:R") (at 40.64 161.29 180) (unit 1)
     (in_bom yes) (on_board yes) (dnp no) (fields_autoplaced)
-    (property "Reference" "R12" (at 43.18 160.02 0)
+    (property "Reference" "R16" (at 43.18 160.02 0)
       (effects (font (size 1.27 1.27)) (justify right))
     )
@@
       (project "OpenHand"
         (path "/f1fbd835-8408-4592-854c-2fbec9d052ec/286dde41-8068-419e-b7de-6276970410d8"
-          (reference "R12") (unit 1)
+          (reference "R16") (unit 1)
         )
       )
@@
   (symbol (lib_id "Device:R") (at 124.46 140.97 180) (unit 1)
     (in_bom yes) (on_board yes) (dnp no) (fields_autoplaced)
-    (property "Reference" "R10" (at 127 139.7 0)
+    (property "Reference" "R14" (at 127 139.7 0)
       (effects (font (size 1.27 1.27)) (justify right))
     )
@@
       (project "OpenHand"
         (path "/f1fbd835-8408-4592-854c-2fbec9d052ec/286dde41-8068-419e-b7de-6276970410d8"
-          (reference "R10") (unit 1)
-        )
-      )
-    )
-  )
-  (symbol (lib_id "Amplifier_Instrumentation:INA333xxDGK") (at 73.66 53.34 0) (unit 1)
-    (in_bom yes) (on_board yes) (dnp no) (fields_autoplaced)
-    (property "Reference" "U3" (at 88.9 49.1491 0)
-      (effects (font (size 1.27 1.27)))
-    )
-    (property "Value" "INA333xxDGK" (at 88.9 51.6891 0)
-      (effects (font (size 1.27 1.27)))
-    )
-    (property "Footprint" "Package_SO:VSSOP-8_3.0x3.0mm_P0.65mm" (at 73.66 60.96 0)
-      (effects (font (size 1.27 1.27)) hide)
-    )
-    (property "Datasheet" "https://www.ti.com/lit/ds/symlink/ina333.pdf" (at 76.2 53.34 0)
-      (effects (font (size 1.27 1.27)) hide)
-    )
-    (pin "1")
-    (pin "2")
-    (pin "3")
-    (pin "4")
-    (pin "5")
-    (pin "6")
-    (pin "7")
-    (pin "8")
-    (instances
-      (project "OpenHand"
-        (path "/f1fbd835-8408-4592-854c-2fbec9d052ec/286dde41-8068-419e-b7de-6276970410d8"
-          (reference "U3") (unit 1)
+          (reference "R14") (unit 1)
         )
       )
@@
   (symbol (lib_id "power:Earth") (at 81.28 170.18 0) (unit 1)
     (in_bom yes) (on_board yes) (dnp no) (fields_autoplaced)
-    (property "Reference" "#PWR032" (at 81.28 176.53 0)
+    (property "Reference" "#PWR038" (at 81.28 176.53 0)
       (effects (font (size 1.27 1.27)) hide)
     )
@@
       (project "OpenHand"
         (path "/f1fbd835-8408-4592-854c-2fbec9d052ec/286dde41-8068-419e-b7de-6276970410d8"
-          (reference "#PWR032") (unit 1)
+          (reference "#PWR038") (unit 1)
         )
       )
@@
   (symbol (lib_id "Analog_ADC:ADS1115IDGS") (at 81.28 154.94 0) (unit 1)
     (in_bom yes) (on_board yes) (dnp no)
-    (property "Reference" "U6" (at 73.66 165.1 0)
+    (property "Reference" "U3" (at 73.66 165.1 0)
       (effects (font (size 1.27 1.27)) (justify left))
     )
@@
       (project "OpenHand"
         (path "/f1fbd835-8408-4592-854c-2fbec9d052ec/286dde41-8068-419e-b7de-6276970410d8"
-          (reference "U6") (unit 1)
+          (reference "U3") (unit 1)
         )
       )
@@
   (symbol (lib_id "power:Earth") (at 40.64 170.18 0) (unit 1)
     (in_bom yes) (on_board yes) (dnp no) (fields_autoplaced)
-    (property "Reference" "#PWR031" (at 40.64 176.53 0)
+    (property "Reference" "#PWR037" (at 40.64 176.53 0)
       (effects (font (size 1.27 1.27)) hide)
     )
@@
       (project "OpenHand"
         (path "/f1fbd835-8408-4592-854c-2fbec9d052ec/286dde41-8068-419e-b7de-6276970410d8"
-          (reference "#PWR031") (unit 1)
+          (reference "#PWR037") (unit 1)
         )
       )
@@
   (symbol (lib_id "power:+3V3") (at 93.98 121.92 0) (unit 1)
     (in_bom yes) (on_board yes) (dnp no)
-    (property "Reference" "#PWR030" (at 93.98 125.73 0)
+    (property "Reference" "#PWR036" (at 93.98 125.73 0)
       (effects (font (size 1.27 1.27)) hide)
     )
@@
       (project "OpenHand"
         (path "/f1fbd835-8408-4592-854c-2fbec9d052ec/286dde41-8068-419e-b7de-6276970410d8"
-          (reference "#PWR030") (unit 1)
-        )
-      )
-    )
-  )
-  (symbol (lib_id "Amplifier_Operational:OPA333xxDBV") (at 73.66 78.74 0) (unit 1)
-    (in_bom yes) (on_board yes) (dnp no) (fields_autoplaced)
-    (property "Reference" "U5" (at 86.36 74.5491 0)
-      (effects (font (size 1.27 1.27)))
-    )
-    (property "Value" "OPA333xxDBV" (at 86.36 77.0891 0)
-      (effects (font (size 1.27 1.27)))
-    )
-    (property "Footprint" "Package_TO_SOT_SMD:SOT-23-5" (at 71.12 83.82 0)
-      (effects (font (size 1.27 1.27)) (justify left) hide)
-    )
-    (property "Datasheet" "http://www.ti.com/lit/ds/symlink/opa333.pdf" (at 73.66 73.66 0)
-      (effects (font (size 1.27 1.27)) hide)
-    )
-    (pin "2")
-    (pin "5")
-    (pin "1")
-    (pin "3")
-    (pin "4")
-    (instances
-      (project "OpenHand"
-        (path "/f1fbd835-8408-4592-854c-2fbec9d052ec/286dde41-8068-419e-b7de-6276970410d8"
-          (reference "U5") (unit 1)
+          (reference "#PWR036") (unit 1)
         )
       )
@@
   (symbol (lib_id "Device:R") (at 93.98 140.97 180) (unit 1)
     (in_bom yes) (on_board yes) (dnp no) (fields_autoplaced)
-    (property "Reference" "R8" (at 96.52 139.7 0)
+    (property "Reference" "R12" (at 96.52 139.7 0)
       (effects (font (size 1.27 1.27)) (justify right))
     )
@@
       (project "OpenHand"
         (path "/f1fbd835-8408-4592-854c-2fbec9d052ec/286dde41-8068-419e-b7de-6276970410d8"
-          (reference "R8") (unit 1)
+          (reference "R12") (unit 1)
         )
       )
@@
   (symbol (lib_id "Device:R") (at 116.84 140.97 180) (unit 1)
     (in_bom yes) (on_board yes) (dnp no) (fields_autoplaced)
-    (property "Reference" "R9" (at 119.38 139.7 0)
+    (property "Reference" "R13" (at 119.38 139.7 0)
       (effects (font (size 1.27 1.27)) (justify right))
     )
@@
       (project "OpenHand"
         (path "/f1fbd835-8408-4592-854c-2fbec9d052ec/286dde41-8068-419e-b7de-6276970410d8"
-          (reference "R9") (unit 1)
+          (reference "R13") (unit 1)
         )
       )
@@
   (symbol (lib_id "Device:R") (at 40.64 146.05 180) (unit 1)
     (in_bom yes) (on_board yes) (dnp no) (fields_autoplaced)
-    (property "Reference" "R11" (at 43.18 144.78 0)
+    (property "Reference" "R15" (at 43.18 144.78 0)
       (effects (font (size 1.27 1.27)) (justify right))
     )
@@
       (project "OpenHand"
         (path "/f1fbd835-8408-4592-854c-2fbec9d052ec/286dde41-8068-419e-b7de-6276970410d8"
-          (reference "R11") (unit 1)
-        )
-      )
-    )
-  )
-  (symbol (lib_id "Amplifier_Operational:OPA333xxDBV") (at 111.76 55.88 0) (unit 1)
-    (in_bom yes) (on_board yes) (dnp no) (fields_autoplaced)
-    (property "Reference" "U4" (at 124.46 51.6891 0)
-      (effects (font (size 1.27 1.27)))
-    )
-    (property "Value" "OPA333xxDBV" (at 124.46 54.2291 0)
-      (effects (font (size 1.27 1.27)))
-    )
-    (property "Footprint" "Package_TO_SOT_SMD:SOT-23-5" (at 109.22 60.96 0)
-      (effects (font (size 1.27 1.27)) (justify left) hide)
-    )
-    (property "Datasheet" "http://www.ti.com/lit/ds/symlink/opa333.pdf" (at 111.76 50.8 0)
-      (effects (font (size 1.27 1.27)) hide)
-    )
-    (pin "2")
-    (pin "5")
-    (pin "1")
-    (pin "3")
-    (pin "4")
-    (instances
-      (project "OpenHand"
-        (path "/f1fbd835-8408-4592-854c-2fbec9d052ec/286dde41-8068-419e-b7de-6276970410d8"
-          (reference "U4") (unit 1)
-        )
-      )
+          (reference "R15") (unit 1)
+        )
+      )

Commit message: Update schematic a bit
Parts:
- renumbered U3 to U5
Changed lines of the file:
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@@
   (symbol (lib_id "power:Earth") (at 81.28 170.18 0) (unit 1)
     (in_bom yes) (on_board yes) (dnp no) (fields_autoplaced)
-    (property "Reference" "#PWR038" (at 81.28 176.53 0)
+    (property "Reference" "#PWR039" (at 81.28 176.53 0)
       (effects (font (size 1.27 1.27)) hide)
     )
@@
       (project "OpenHand"
         (path "/f1fbd835-8408-4592-854c-2fbec9d052ec/286dde41-8068-419e-b7de-6276970410d8"
-          (reference "#PWR038") (unit 1)
+          (reference "#PWR039") (unit 1)
         )
       )
@@
   (symbol (lib_id "Analog_ADC:ADS1115IDGS") (at 81.28 154.94 0) (unit 1)
     (in_bom yes) (on_board yes) (dnp no)
-    (property "Reference" "U3" (at 73.66 165.1 0)
+    (property "Reference" "U5" (at 73.66 165.1 0)
       (effects (font (size 1.27 1.27)) (justify left))
     )
@@
       (project "OpenHand"
         (path "/f1fbd835-8408-4592-854c-2fbec9d052ec/286dde41-8068-419e-b7de-6276970410d8"
-          (reference "U3") (unit 1)
+          (reference "U5") (unit 1)
         )
       )
@@
   (symbol (lib_id "power:Earth") (at 40.64 170.18 0) (unit 1)
     (in_bom yes) (on_board yes) (dnp no) (fields_autoplaced)
-    (property "Reference" "#PWR037" (at 40.64 176.53 0)
+    (property "Reference" "#PWR038" (at 40.64 176.53 0)
       (effects (font (size 1.27 1.27)) hide)
     )
@@
       (project "OpenHand"
         (path "/f1fbd835-8408-4592-854c-2fbec9d052ec/286dde41-8068-419e-b7de-6276970410d8"
-          (reference "#PWR037") (unit 1)
+          (reference "#PWR038") (unit 1)
         )
       )
@@
   (symbol (lib_id "power:+3V3") (at 93.98 121.92 0) (unit 1)
     (in_bom yes) (on_board yes) (dnp no)
-    (property "Reference" "#PWR036" (at 93.98 125.73 0)
+    (property "Reference" "#PWR037" (at 93.98 125.73 0)
       (effects (font (size 1.27 1.27)) hide)
     )
@@
       (project "OpenHand"
         (path "/f1fbd835-8408-4592-854c-2fbec9d052ec/286dde41-8068-419e-b7de-6276970410d8"
-          (reference "#PWR036") (unit 1)
+          (reference "#PWR037") (unit 1)
         )
       )

Commit message: Update sch and board design
Parts:
- added C15, C16: 100n, Capacitor_SMD:C_1206_3216Metric_Pad1.33x1.80mm_HandSolder, symbol Device:C
- added C17, C18, C19, C20, C21, C22: 470n, Capacitor_SMD:C_0805_2012Metric_Pad1.18x1.45mm_HandSolder, symbol Device:C
- added C23, C24: 330n, Capacitor_SMD:C_0805_2012Metric_Pad1.18x1.45mm_HandSolder, symbol Device:C
- added C25, C26: 10u, Capacitor_SMD:C_0805_2012Metric_Pad1.18x1.45mm_HandSolder, symbol Device:C_Polarized
- added D5, D6: SS14, Diode_SMD:D_SOD-123, symbol Device:D_Schottky
- added R18, R19, R28, R30, R38, R39: 47k, Resistor_SMD:R_0805_2012Metric_Pad1.20x1.40mm_HandSolder, symbol Device:R
- added R20, R21, R29, R31: 15k, Resistor_SMD:R_0805_2012Metric_Pad1.20x1.40mm_HandSolder, symbol Device:R
- added R22, R23, R24, R25, R26, R27, R36, R37, R40, R41: 1k, Resistor_SMD:R_0805_2012Metric_Pad1.20x1.40mm_HandSolder, symbol Device:R
- added R32, R33, R42, R43: 10k, Resistor_SMD:R_0805_2012Metric_Pad1.20x1.40mm_HandSolder, symbol Device:R
- added R34, R35, R44, R45, R46, R47: 18k, Resistor_SMD:R_0805_2012Metric_Pad1.20x1.40mm_HandSolder, symbol Device:R
- added RV4, RV5: 100k, Potentiometer_SMD:Potentiometer_Vishay_TS53YJ_Vertical, symbol Device:R_Potentiometer
- added TP44: TP_HALL_01, TestPoint:TestPoint_Pad_D1.0mm, symbol Connector:TestPoint
- added TP44: TP_BATT_SENSE, TestPoint:TestPoint_Pad_D1.0mm, symbol Connector:TestPoint
- added TP44: TP_ADC_RDY, TestPoint:TestPoint_Pad_D1.0mm, symbol Connector:TestPoint
- added TP44: TP_HALL_03, TestPoint:TestPoint_Pad_D1.0mm, symbol Connector:TestPoint
- added TP44: TP_HALL_02, TestPoint:TestPoint_Pad_D1.0mm, symbol Connector:TestPoint
- added U6, U7: LM324, Package_SO:SO-14_5.3x10.2mm_P1.27mm, symbol Amplifier_Operational:LM324
- R48: renamed from R12; footprint Resistor_SMD:R_1206_3216Metric -> Resistor_SMD:R_0805_2012Metric_Pad1.20x1.40mm_HandSolder
- R49: renamed from R13; footprint Resistor_SMD:R_1206_3216Metric -> Resistor_SMD:R_0805_2012Metric_Pad1.20x1.40mm_HandSolder
- R50: renamed from R14; footprint Resistor_SMD:R_1206_3216Metric -> Resistor_SMD:R_0805_2012Metric_Pad1.20x1.40mm_HandSolder
- R51: renamed from R15; footprint Resistor_SMD:R_1206_3216Metric -> Resistor_SMD:R_0805_2012Metric_Pad1.20x1.40mm_HandSolder
- R52: renamed from R16; footprint Resistor_SMD:R_1206_3216Metric -> Resistor_SMD:R_0805_2012Metric_Pad1.20x1.40mm_HandSolder
- renumbered U5 to U8
Connections:
- net ADC_ALERT_RDY: now also TP44.1
- net Earth: now also C15.2, C16.2, C23.1, C24.1, C25.2, C26.2, R18.1, R19.1, R29.2, R31.2, R34.2, R35.2, R40.2, R41.2, R44.2, R45.2, R46.2, R47.2
- net HALL_SENS_01_S: now also TP44.1
- net HALL_SENS_02_S: now also TP44.1
- net HALL_SENS_03_S: now also TP44.1
- net at R51.1, R52.2, U8.4 (AIN0): now also TP44.1
- net BAT_P renamed +BATT
- new net: C21.2, R42.2, U7.12 (+), U7.8
- new net: R40.1, RV4.3, U7.13 (-)
- new net: D5.2 (A), R38.1, U7.14
- new net: R41.1, RV5.3, U6.13 (-)
- new net: C23.2, R36.2, U7.10 (+)
- new net: C24.2, R37.2, U6.10 (+)
- new net: C22.2, R43.2, U6.12 (+), U6.8
- new net: R43.1, R47.1, U6.9 (-)
- new net: R42.1, R46.1, U7.9 (-)
- new net: R21.2, R27.1, R33.2, U6.7
- new net: R33.1, R35.1, U6.6 (-)
- new net: D6.2 (A), R39.1, U6.14
- new net: C17.1, R28.2, U7.1
- new net: R24.1, R28.1, U7.2 (-)
- new net: R18.2, R22.1, U7.3 (+)
- new net: C20.2, R31.1, U6.5 (+)
- new net: C17.2, C18.1, R20.1
- new net: C18.2, R29.1, U7.5 (+)
- new net: C19.1, R30.2, U6.1
- new net: R25.1, R30.1, U6.2 (-)
- new net: R19.2, R23.1, U6.3 (+)
- new net: R39.2, RV5.1, RV5.2
- new net: R20.2, R26.1, R32.2, U7.7
- new net: R32.1, R34.1, U7.6 (-)
- new net: C19.2, C20.1, R21.1
- new net: R38.2, RV4.1, RV4.2
- new net +5V: C15.1, C16.1, U6.4 (V+), U7.4 (V+)
- new net -5V: U6.11 (V-), U7.11 (V-)
- new net EMG_1_MIDPOINT: C22.1, R27.2, R37.1
- new net EMG_1_N: R25.2
- new net EMG_1_P: R23.2
- new net EMG_1_UC: C26.1, D6.1 (K), R45.1
- new net EMG_2_MIDPOINT: C21.1, R26.2, R36.1
- new net EMG_2_N: R24.2
- new net EMG_2_P: R22.2
- new net EMG_2_UC: C25.1, D5.1 (K), R44.1
Other:
- note added: "(OpenEMG project by charleslabs.fr)"
- note added: "Differential amplifier"
- note added: "High-pass filter"
- note added: "Low-pass filter"
- note added: "TODO: add testpoints here!"
- note added: "Tunable amplifier"
- note removed: "Hall effect sensors supply"
- moved on the sheet: R48, R49, R50, R51, R52, U8

Commit message: Update schm
Parts:
- removed R49, R50: 10k, Resistor_SMD:R_0805_2012Metric_Pad1.20x1.40mm_HandSolder, symbol Device:R
- removed TP44: TP_HALL_01, TestPoint:TestPoint_Pad_D1.0mm, symbol Connector:TestPoint
- removed TP44: TP_BATT_SENSE, TestPoint:TestPoint_Pad_D1.0mm, symbol Connector:TestPoint
- removed TP44: TP_ADC_RDY, TestPoint:TestPoint_Pad_D1.0mm, symbol Connector:TestPoint
- removed TP44: TP_HALL_03, TestPoint:TestPoint_Pad_D1.0mm, symbol Connector:TestPoint
- removed TP44: TP_HALL_02, TestPoint:TestPoint_Pad_D1.0mm, symbol Connector:TestPoint
- added JP9: JMPR_I2C_ADC_SDA, Jumper:SolderJumper-2_P1.3mm_Bridged_RoundedPad1.0x1.5mm, symbol Jumper:SolderJumper_2_Bridged
- added JP9: JMPR_EMG_2_UC, Jumper:SolderJumper-2_P1.3mm_Bridged_RoundedPad1.0x1.5mm, symbol Jumper:SolderJumper_2_Bridged
- added JP9: JMPR_I2C_ADC_SCL, Jumper:SolderJumper-2_P1.3mm_Bridged_RoundedPad1.0x1.5mm, symbol Jumper:SolderJumper_2_Bridged
- added JP9: JMPR_EMG_1_UC, Jumper:SolderJumper-2_P1.3mm_Bridged_RoundedPad1.0x1.5mm, symbol Jumper:SolderJumper_2_Bridged
- added TP50: TP_EMG_1_HP, symbol Connector:TestPoint_Small
- added TP50: TP_HALL_03, symbol Connector:TestPoint_Small
- added TP50: TP_HALL_02, symbol Connector:TestPoint_Small
- added TP50: TP_BATT_SENSE, symbol Connector:TestPoint_Small
- added TP50: TP_ADC_RDY, symbol Connector:TestPoint_Small
- added TP50: TP_EMG_1_LP, symbol Connector:TestPoint_Small
- added TP50: TP_EMG_2_LP, symbol Connector:TestPoint_Small
- added TP50: TP_EMG_2_UC, symbol Connector:TestPoint_Small
- added TP50: TP_EMG_1_UC, symbol Connector:TestPoint_Small
- added TP50: TP_EMG_2_HP, symbol Connector:TestPoint_Small
- added TP50: TP_EMG_1_AMP, symbol Connector:TestPoint_Small
- added TP50: TP_EMG_2_AMP, symbol Connector:TestPoint_Small
- added TP50: TP_HALL_01, symbol Connector:TestPoint_Small
- renumbered R18 to R20, R19 to R21, R20 to R22, R21 to R23, R22 to R24, R23 to R25, R24 to R26, R25 to R27, R26 to R28, R27 to R29, R28 to R30, R29 to R31, R30 to R32, R31 to R33, R32 to R34, R33 to R35, R34 to R36, R35 to R37, R36 to R38, R37 to R39, R38 to R40, R39 to R41, R40 to R42, R41 to R43, R42 to R44, R43 to R45, R44 to R46, R45 to R47, R46 to R48, R47 to R49, R48 to R50, R51 to R53, R52 to R54
Connections:
- net ADC_ALERT_RDY: now also TP50.1
- net EMG_1_MIDPOINT: now also TP50.1
- net EMG_1_UC: now also JP9.2 (B), TP50.1; no longer C26.1, D6.1 (K), R47.1
- net EMG_2_MIDPOINT: now also TP50.1
- net EMG_2_UC: now also JP9.2 (B), TP50.1; no longer C25.1, D5.1 (K), R46.1
- net HALL_SENS_01_S: now also TP50.1
- net HALL_SENS_02_S: now also TP50.1
- net HALL_SENS_03_S: now also TP50.1
- net UC_SCL: now also JP9.2 (B); no longer U8.10 (SCL)
- net UC_SDA: now also JP9.1 (A); no longer U8.9 (SDA)
- net at C21.2, R44.2, U7.12 (+)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: now also TP50.1
- net at C22.2, R45.2, U6.12 (+)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: now also TP50.1
- net at R53.1, R54.2, U8.4 (AIN0): now also TP50.1
- net at C17.1, R30.2, U7.1: now also TP50.1
- net at C19.1, R32.2, U6.1: now also TP50.1
- new net: C25.1, D5.1 (K), JP9.1 (A), R46.1
- new net: C26.1, D6.1 (K), JP9.1 (A), R47.1
- new net: JP9.2 (B), U8.9 (SDA)
- new net: JP9.1 (A), U8.10 (SCL)
Other:
- note removed: "I2C pullups"
- note removed: "TODO: add testpoints here!"
- moved on the sheet: C17, C19, C20, C23, C24, C25, C26, D5, D6, R26, R27, R40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
