File: hardware/OpenHand/OpenHand.kicad_sch (KiCad schematic)
At the start: 52 parts, among them J1 CONN_MOTOR_1, J10 CONN_JTAG, J11 CONN_FDBK_2, J12 CONN_EMG_2, J13 CONN_POS_3, J2 CONN_MOTOR_2, J3 CONN_BATT, J4 USB_C_CONN, J5 CONN_POS_1, J6 CONN_MOTOR_3, J7 CONN_FDBK_1, J8 CONN_EMG_1, J9 CONN_POS_2, Q1 2N7002, Q2 2N7002, SW1 SW_Push, SW2 BTN_RST, SW3 BTN_BOOT, U1 CH340C, U2 STM32F103RETx

Commit message: Update sch and board design
Parts:
- added JP9: JMPR_RST, Jumper:SolderJumper-2_P1.3mm_Bridged_RoundedPad1.0x1.5mm, symbol Jumper:SolderJumper_2_Bridged
- added JP9: JMPR_BTN_BOOT, Jumper:SolderJumper-2_P1.3mm_Bridged_RoundedPad1.0x1.5mm, symbol Jumper:SolderJumper_2_Bridged
- added JP9: JMPR_LED_2, Jumper:SolderJumper-2_P1.3mm_Bridged_RoundedPad1.0x1.5mm, symbol Jumper:SolderJumper_2_Bridged
- added JP9: JMPR_POT_1, Jumper:SolderJumper-2_P1.3mm_Bridged_RoundedPad1.0x1.5mm, symbol Jumper:SolderJumper_2_Bridged
- added JP9: JMPR_BOOT, Jumper:SolderJumper-2_P1.3mm_Bridged_RoundedPad1.0x1.5mm, symbol Jumper:SolderJumper_2_Bridged
- added JP9: JMPR_TRIM_1, Jumper:SolderJumper-2_P1.3mm_Bridged_RoundedPad1.0x1.5mm, symbol Jumper:SolderJumper_2_Bridged
- added JP9: JMPR_TRIM_2, Jumper:SolderJumper-2_P1.3mm_Bridged_RoundedPad1.0x1.5mm, symbol Jumper:SolderJumper_2_Bridged
- added JP9: JMPR_BTN_RST, Jumper:SolderJumper-2_P1.3mm_Bridged_RoundedPad1.0x1.5mm, symbol Jumper:SolderJumper_2_Bridged
- added JP9: JMPR_USB_P, Jumper:SolderJumper-2_P1.3mm_Bridged_RoundedPad1.0x1.5mm, symbol Jumper:SolderJumper_2_Bridged
- added JP9: JMPR_TX, Jumper:SolderJumper-2_P1.3mm_Bridged_RoundedPad1.0x1.5mm, symbol Jumper:SolderJumper_2_Bridged
- added JP9: JMPR_USB_N, Jumper:SolderJumper-2_P1.3mm_Bridged_RoundedPad1.0x1.5mm, symbol Jumper:SolderJumper_2_Bridged
- added JP9: JMPR_LED_1, Jumper:SolderJumper-2_P1.3mm_Bridged_RoundedPad1.0x1.5mm, symbol Jumper:SolderJumper_2_Bridged
- added JP9: JMPR_RX, Jumper:SolderJumper-2_P1.3mm_Bridged_RoundedPad1.0x1.5mm, symbol Jumper:SolderJumper_2_Bridged
- added JP9: JMPR_BTN_1, Jumper:SolderJumper-2_P1.3mm_Bridged_RoundedPad1.0x1.5mm, symbol Jumper:SolderJumper_2_Bridged
- added TP1: TP_UC_RST, TestPoint:TestPoint_Pad_D1.0mm, symbol Connector:TestPoint
- added TP10: TP_HW_REV_2, TestPoint:TestPoint_Pad_D1.0mm, symbol Connector:TestPoint
- added TP11: TP_HW_REV_1, TestPoint:TestPoint_Pad_D1.0mm, symbol Connector:TestPoint
- added TP12: TP_LED_1, TestPoint:TestPoint_Pad_D1.0mm, symbol Connector:TestPoint
- added TP13: TP_HW_REV_3, TestPoint:TestPoint_Pad_D1.0mm, symbol Connector:TestPoint
- added TP14: TP_BTN_1, TestPoint:TestPoint_Pad_D1.0mm, symbol Connector:TestPoint
- added TP15: TP_LED_2, TestPoint:TestPoint_Pad_D1.0mm, symbol Connector:TestPoint
- added TP16: TP_HW_REV_4, TestPoint:TestPoint_Pad_D1.0mm, symbol Connector:TestPoint
- added TP2: TP_UC_RX, TestPoint:TestPoint_Pad_D1.0mm, symbol Connector:TestPoint
- added TP3: TP_UC_TX, TestPoint:TestPoint_Pad_D1.0mm, symbol Connector:TestPoint
- added TP4: TP_USB_D_P, TestPoint:TestPoint_Pad_D1.0mm, symbol Connector:TestPoint
- added TP5: TP_USB_D_N, TestPoint:TestPoint_Pad_D1.0mm, symbol Connector:TestPoint
- added TP6: TP_UC_BOOT, TestPoint:TestPoint_Pad_D1.0mm, symbol Connector:TestPoint
- added TP7: TP_TRIM_POT_1, TestPoint:TestPoint_Pad_D1.0mm, symbol Connector:TestPoint
- added TP8: TP_TRIM_POT_2, TestPoint:TestPoint_Pad_D1.0mm, symbol Connector:TestPoint
- added TP9: TP_POT_1, TestPoint:TestPoint_Pad_D1.0mm, symbol Connector:TestPoint
- C1, C2, C3, C4: footprint Capacitor_SMD:C_1206_3216Metric -> Capacitor_SMD:C_1206_3216Metric_Pad1.33x1.80mm_HandSolder
- J1, J11, J2, J3, J6, J7: footprint (none) -> Connector_JST:JST_EH_S2B-EH_1x02_P2.50mm_Horizontal
- J10: footprint (none) -> Connector_PinHeader_2.54mm:PinHeader_1x06_P2.54mm_Vertical
- J12, J13, J5, J8, J9: footprint (none) -> Connector_JST:JST_EH_S3B-EH_1x03_P2.50mm_Horizontal
- R1, R10, R2, R5, R6, R7, R8: footprint Resistor_SMD:R_1206_3216Metric -> Resistor_SMD:R_0805_2012Metric_Pad1.20x1.40mm_HandSolder
- R11, R9: value 1k -> 4k7; footprint Resistor_SMD:R_1206_3216Metric -> Resistor_SMD:R_0805_2012Metric_Pad1.20x1.40mm_HandSolder
- R3, R4: footprint (none) -> Resistor_SMD:R_0805_2012Metric_Pad1.20x1.40mm_HandSolder
- RV1, RV2, RV3: footprint (none) -> Potentiometer_SMD:Potentiometer_Vishay_TS53YJ_Vertical
- SW1, SW2, SW3: footprint (none) -> Button_Switch_SMD:SW_Tactile_SPST_NO_Straight_CK_PTS636Sx25SMTRLFS
Connections:
- net HALL_SENS_01_P is gone; now on net +3V3: J5.3 (Pin_3)
- net HALL_SENS_02_P is gone; now on net +3V3: J9.3 (Pin_3)
- net HALL_SENS_03_P is gone; now on net +3V3: J13.3 (Pin_3)
- net BTN_1: now also JP9.2 (B); no longer R10.2, SW1.1
- net HW_REV_1: now also TP11.1
- net HW_REV_2: now also TP10.1
- net HW_REV_3: now also TP13.1
- net HW_REV_4: now also TP16.1
- net LED_1: now also JP9.2 (B); no longer D1.2 (A)
- net LED_2: now also JP9.2 (B); no longer D2.2 (A)
- net POT_1: now also JP9.2 (B); no longer RV3.2
- net TRIM_POT_1: now also JP9.2 (B); no longer RV1.2
- net TRIM_POT_2: now also JP9.2 (B); no longer RV2.2
- net UC_BOOT: now also JP9.2 (B), JP9.2 (B); no longer C4.1, Q2.3 (D), SW3.1
- net UC_RST: now also JP9.2 (B), JP9.2 (B); no longer C3.1, Q1.3 (D), SW2.1
- net UC_RX: now also JP9.2 (B); no longer U1.2 (TXD)
- net UC_TX: now also JP9.1 (A); no longer U1.3 (RXD)
- net USB_D_N: now also JP9.2 (B), TP5.1; no longer U1.6 (UD-)
- net USB_D_P: now also JP9.1 (A), TP4.1; no longer U1.5 (UD+)
- net +BATT renamed BAT_P
- new net: C3.1, JP9.1 (A), Q1.3 (D), TP1.1
- new net: JP9.1 (A), RV3.2, TP9.1
- new net: JP9.1 (A), SW3.1
- new net: JP9.1 (A), SW2.1
- new net: D2.2 (A), JP9.1 (A), TP15.1
- new net: D1.2 (A), JP9.1 (A), TP12.1
- new net: C4.1, JP9.1 (A), Q2.3 (D), TP6.1
- new net: JP9.1 (A), TP2.1, U1.2 (TXD)
- new net: JP9.2 (B), TP3.1, U1.3 (RXD)
- new net: JP9.2 (B), U1.5 (UD+)
- new net: JP9.1 (A), U1.6 (UD-)
- new net: JP9.1 (A), R10.2, SW1.1, TP14.1
- new net: JP9.1 (A), RV1.2, TP7.1
- new net: JP9.1 (A), RV2.2, TP8.1
Other:
- sheet PSU, Charger renamed PSU
- note added: "TODO: add testpoints here!"
- note added: "TODO: research what pins should be connected to what function"
- moved on the sheet: C3, C4, D1, D2, Q1, Q2, R10, R11, R3, R4, R9, RV1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

Commit message: Update schm
Parts:
- removed TP1: TP_UC_RST, TestPoint:TestPoint_Pad_D1.0mm, symbol Connector:TestPoint
- removed TP10: TP_HW_REV_2, TestPoint:TestPoint_Pad_D1.0mm, symbol Connector:TestPoint
- removed TP11: TP_HW_REV_1, TestPoint:TestPoint_Pad_D1.0mm, symbol Connector:TestPoint
- removed TP12: TP_LED_1, TestPoint:TestPoint_Pad_D1.0mm, symbol Connector:TestPoint
- removed TP13: TP_HW_REV_3, TestPoint:TestPoint_Pad_D1.0mm, symbol Connector:TestPoint
- removed TP14: TP_BTN_1, TestPoint:TestPoint_Pad_D1.0mm, symbol Connector:TestPoint
- removed TP15: TP_LED_2, TestPoint:TestPoint_Pad_D1.0mm, symbol Connector:TestPoint
- removed TP16: TP_HW_REV_4, TestPoint:TestPoint_Pad_D1.0mm, symbol Connector:TestPoint
- removed TP2: TP_UC_RX, TestPoint:TestPoint_Pad_D1.0mm, symbol Connector:TestPoint
- removed TP3: TP_UC_TX, TestPoint:TestPoint_Pad_D1.0mm, symbol Connector:TestPoint
- removed TP4: TP_USB_D_P, TestPoint:TestPoint_Pad_D1.0mm, symbol Connector:TestPoint
- removed TP5: TP_USB_D_N, TestPoint:TestPoint_Pad_D1.0mm, symbol Connector:TestPoint
- removed TP6: TP_UC_BOOT, TestPoint:TestPoint_Pad_D1.0mm, symbol Connector:TestPoint
- removed TP7: TP_TRIM_POT_1, TestPoint:TestPoint_Pad_D1.0mm, symbol Connector:TestPoint
- removed TP8: TP_TRIM_POT_2, TestPoint:TestPoint_Pad_D1.0mm, symbol Connector:TestPoint
- removed TP9: TP_POT_1, TestPoint:TestPoint_Pad_D1.0mm, symbol Connector:TestPoint
- added R12, R13, R51, R52: 10k, Resistor_SMD:R_0805_2012Metric_Pad1.20x1.40mm_HandSolder, symbol Device:R
- added TP34: TP_USB_D_N, symbol Connector:TestPoint_Small
- added TP34: TP_UC_TX, symbol Connector:TestPoint_Small
- added TP50 (x2): TP_UC_PIN_XX, symbol Connector:TestPoint_Small
- added TP50: TP_USB_D_P, symbol Connector:TestPoint_Small
- added TP50: TP_HW_REV_1, symbol Connector:TestPoint_Small
- added TP50: TP_UC_RX, symbol Connector:TestPoint_Small
- added TP50: TP_UC_BOOT, symbol Connector:TestPoint_Small
- added TP50: TP_UC_RST, symbol Connector:TestPoint_Small
- added TP50: TP_UC_SDA, symbol Connector:TestPoint_Small
- added TP50: TP_POT_1, symbol Connector:TestPoint_Small
- added TP50: TP_HW_REV_2, symbol Connector:TestPoint_Small
- added TP50: TP_UC_SCL, symbol Connector:TestPoint_Small
- added TP50: TP_LED_2, symbol Connector:TestPoint_Small
- added TP50: TP_BTN_1, symbol Connector:TestPoint_Small
- added TP50: TP_TRIM_POT_1, symbol Connector:TestPoint_Small
- added TP50: TP_TRIM_POT_2, symbol Connector:TestPoint_Small
- added TP50: TP_LED_1, symbol Connector:TestPoint_Small
- added TP50: TP_HW_REV_3, symbol Connector:TestPoint_Small
- added TP50: TP_HW_REV_4, symbol Connector:TestPoint_Small
- renumbered JP1 to JP10, JP2 to JP11, JP3 to JP12, JP4 to JP13, JP5 to JP15, JP6 to JP16, JP7 to JP17, JP8 to JP18, RV3 to RV1, RV1 to RV2, RV2 to RV3
Connections:
- net +3V3: now also R12.1, R13.1
- net HW_REV_1: now also TP50.1
- net HW_REV_2: now also TP50.1
- net HW_REV_3: now also TP50.1
- net HW_REV_4: now also TP50.1
- net USB_D_N: now also TP34.1
- net USB_D_P: now also TP50.1
- net at C3.1, JP9.1 (A), Q1.3 (D): now also TP50.1
- net at JP9.1 (A), RV1.2: now also TP50.1
- net at JP9.1 (A), SW3.1: now also R13.2
- net at JP9.1 (A), SW2.1: now also R12.2
- net at D2.2 (A), JP9.1 (A): now also TP50.1
- net at D1.2 (A), JP9.1 (A): now also TP50.1
- net at C4.1, JP9.1 (A), Q2.3 (D): now also TP50.1
- net at JP9.1 (A), R10.2, SW1.1: now also TP50.1
- net at JP9.1 (A), RV2.2: now also TP50.1
- net at JP9.1 (A), RV3.2: now also TP50.1
Other:
- note added: "I2C pullups"
- moved on the sheet: J4, JP10, JP11, JP12, JP13, JP15, JP16, JP17, JP18, JP9, R1, R2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

Commit message: Update schm and pcb
Parts:
- RV1: value POT_1 -> TRIM_POT_3
- renumbered R12 to R14, R13 to R15
Connections:
- net POT_1 renamed TRIM_POT_3
Other:
- moved on the sheet: JP9, RV1, RV3, TP50

Commit message: Update schm and pcb
Parts:
- removed TP50: TP_POT_1, symbol Connector:TestPoint_Small
- removed TP50: TP_BTN_1, symbol Connector:TestPoint_Small
- removed TP50: TP_TRIM_POT_1, symbol Connector:TestPoint_Small
- removed TP50: TP_TRIM_POT_2, symbol Connector:TestPoint_Small
- added TP50: TP_UC_PIN_PC15, TestPoint:TestPoint_Pad_D1.0mm, symbol Connector:TestPoint_Small
- added TP50: TP_UC_PIN_PC0, TestPoint:TestPoint_Pad_D1.0mm, symbol Connector:TestPoint_Small
- added TP50: TP_UC_PIN_PC3, TestPoint:TestPoint_Pad_D1.0mm, symbol Connector:TestPoint_Small
- added TP50: TP_UC_PIN_PD2, TestPoint:TestPoint_Pad_D1.0mm, symbol Connector:TestPoint_Small
- added TP50: TP_UC_PIN_PB5, TestPoint:TestPoint_Pad_D1.0mm, symbol Connector:TestPoint_Small
- added TP50: TP_UC_PIN_PB10, TestPoint:TestPoint_Pad_D1.0mm, symbol Connector:TestPoint_Small
- added TP50: TP_UC_PIN_PD0, TestPoint:TestPoint_Pad_D1.0mm, symbol Connector:TestPoint_Small
- added TP50: TP_UC_PIN_PB11, TestPoint:TestPoint_Pad_D1.0mm, symbol Connector:TestPoint_Small
- added TP50: TP_UC_PIN_PD1, TestPoint:TestPoint_Pad_D1.0mm, symbol Connector:TestPoint_Small
- added TP50: TP_UC_PIN_PC1, TestPoint:TestPoint_Pad_D1.0mm, symbol Connector:TestPoint_Small
- added TP50: TP_UC_PIN_PC2, TestPoint:TestPoint_Pad_D1.0mm, symbol Connector:TestPoint_Small
- added TP50: TP_UC_PIN_PB2, TestPoint:TestPoint_Pad_D1.0mm, symbol Connector:TestPoint_Small
- TP34, TP50: footprint (none) -> TestPoint:TestPoint_Pad_D1.0mm
- TP50: value TP_UC_PIN_XX -> TP_UC_PIN_PC14; footprint (none) -> TestPoint:TestPoint_Pad_D1.0mm
- TP50: value TP_UC_SDA -> TP_UC_SCL; footprint (none) -> TestPoint:TestPoint_Pad_D1.0mm
- TP50: value TP_UC_SCL -> TP_UC_SDA; footprint (none) -> TestPoint:TestPoint_Pad_D1.0mm
- TP50: value TP_UC_PIN_XX -> TP_UC_PIN_PC13; footprint (none) -> TestPoint:TestPoint_Pad_D1.0mm
- renumbered R8 to R10, R9 to R11, R10 to R12, R11 to R13, R5 to R7, R6 to R8, R7 to R9
Connections:
- net +3V3: now also R51.2, R52.2, U2.1 (VBAT), U2.13 (VDDA), U2.19 (VDD), U2.32 (VDD), U2.48 (VDD), U2.64 (VDD)
- net EMG_1_UC: now also U2.26 (PB0)
- net EMG_2_UC: now also U2.27 (PB1)
- net Earth: now also U2.12 (VSSA), U2.18 (VSS), U2.31 (VSS), U2.47 (VSS), U2.63 (VSS)
- net FDBK_MOTOR_1_UC1: now also U2.37 (PC6)
- net FDBK_MOTOR_1_UC2: now also U2.39 (PC8)
- net FDBK_MOTOR_2_UC1: now also U2.38 (PC7)
- net FDBK_MOTOR_2_UC2: now also U2.40 (PC9)
- net FDBK_MOTOR_EN: now also U2.36 (PB15)
- net FDBK_MOTOR_FAULT: now also U2.23 (PA7)
- net HW_REV_1: now also U2.14 (PA0)
- net HW_REV_2: now also U2.15 (PA1)
- net HW_REV_3: now also U2.16 (PA2)
- net HW_REV_4: now also U2.17 (PA3)
- net JTAG_RST: now also U2.56 (PB4)
- net JTAG_TCK: now also U2.49 (PA14)
- net JTAG_TDI: now also U2.50 (PA15)
- net JTAG_TDO: now also U2.55 (PB3)
- net JTAG_TMS: now also U2.46 (PA13)
- net LED_1: now also U2.52 (PC11)
- net LED_2: now also U2.53 (PC12)
- net MOTOR_1_EN: now also U2.33 (PB12)
- net MOTOR_1_FAULT: now also U2.20 (PA4)
- net MOTOR_1_UC1: now also U2.41 (PA8)
- net MOTOR_1_UC2: now also U2.44 (PA11)
- net MOTOR_2_EN: now also U2.34 (PB13)
- net MOTOR_2_FAULT: now also U2.21 (PA5)
- net MOTOR_2_UC1: now also U2.42 (PA9)
- net MOTOR_2_UC2: now also U2.45 (PA12)
- net MOTOR_3_EN: now also U2.35 (PB14)
- net MOTOR_3_FAULT: now also U2.22 (PA6)
- net MOTOR_3_UC1: now also U2.43 (PA10)
- net MOTOR_3_UC2: now also U2.51 (PC10)
- net UC_RX: now also TP50.1, U2.59 (PB7)
- net UC_SCL: now also R52.1, TP50.1, U2.61 (PB8)
- net UC_SDA: now also R51.1, TP50.1, U2.62 (PB9)
- net UC_TX: now also TP34.1, U2.58 (PB6)
- net at TP50.1: now also U2.3 (PC14)
- net at TP50.1: now also U2.2 (PC13)
- net at U2.10 (PC2): now also TP50.1
- net at U2.11 (PC3): now also TP50.1
- net ADC_1_ALERT_RDY: now reaches U2.24 (PC4)
- net ADC_2_ALERT_RDY: now reaches U2.25 (PC5)
- net at U2.28 (PB2): now also TP50.1
- net at U2.29 (PB10): now also TP50.1
- net at U2.30 (PB11): now also TP50.1
- net at U2.4 (PC15): now also TP50.1
- net at U2.5 (PD0): now also TP50.1
- net at U2.54 (PD2): now also TP50.1
- net at U2.57 (PB5): now also TP50.1
- net at U2.6 (PD1): now also TP50.1
- net at U2.8 (PC0): now also TP50.1
- net at U2.9 (PC1): now also TP50.1
Other:
- note added: "I2C pullups and test points"
- note added: "PCB design parameters: - min trace width 0.2mm and spacing 0.2mm - via hole size/diameter: 0.3mm / 0.5mm"
- note added: "TODO: - Make a bill of materials (BOM) - Keep as much clearance between traces as possible/available - Add some graphics and logos on silkscreen - Add version somewhere also on siklscreen - Add JLC order number on PCB - Double-check all the footprint sizes and dimensions"
- note added: "UART test points"
- note removed: "- Make sure to add solderable jumpers so we can disconnect parts of the circuits we don't want to test (SolderJumper_2_Bridged) - Use 0805 resistors and capacitors wherever possible (standard values: 1k, 10k...) - Add a lot of test points, and make them somewhat small - Make a good silkscreen that is not cluttered, no need for all component markings. - Watch out for thermals, especially with moto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"
- note removed: "I2C pullups"
- note removed: "PCB manufacturing capabilities: - min trace width 0.2mm and spacing 0.2mm - min via hole size/diameter: 0.3mm / 0.5mm"
- note removed: "TODO: add testpoints here!"
- note removed: "TODO: research what pins should be connected to what function"
- moved on the sheet: R51, R52, TP34, TP50, U2
