File: hardware/OpenHand/OpenHand.kicad_pcb (KiCad board)
At the start: 2 copper layers, 110 x 40 mm, 5 parts, among them U2 STM32F103RETx

Commit message: Minor updates to schm
Parts:
- moved U2 10.5 mm to (130.4, 118.6)
- renumbered He to H2
Connections:
- U2 pad 60: unconnected-(U2-BOOT0-Pad60) -> UC_BOOT
- U2 pad 7: unconnected-(U2-NRST-Pad7) -> UC_RST

Commit message: Update sch and board design
Parts:
- added C1: 1u, Capacitor_SMD:C_1206_3216Metric_Pad1.33x1.80mm_HandSolder, F.Cu at (116.6, 105.6)
- added C10: 10u, Capacitor_SMD:C_0805_2012Metric_Pad1.18x1.45mm_HandSolder, F.Cu at (118.2, 143.4)
- added C11: 10u, Capacitor_SMD:C_0805_2012Metric_Pad1.18x1.45mm_HandSolder, F.Cu at (124.8, 143.4)
- added C12: 100n, Capacitor_SMD:C_1206_3216Metric_Pad1.33x1.80mm_HandSolder, F.Cu at (126.6, 147.0)
- added C13: 22u, Capacitor_SMD:C_0805_2012Metric_Pad1.18x1.45mm_HandSolder, F.Cu at (102.4, 121.6)
- added C14: 22u, Capacitor_SMD:C_0805_2012Metric_Pad1.18x1.45mm_HandSolder, F.Cu at (113.6, 121.6)
- added C15: 100n, Capacitor_SMD:C_1206_3216Metric_Pad1.33x1.80mm_HandSolder, F.Cu at (250.0, 40.6)
- added C16: 100n, Capacitor_SMD:C_1206_3216Metric_Pad1.33x1.80mm_HandSolder, F.Cu at (245.0, 40.3)
- added C17: 470n, Capacitor_SMD:C_0805_2012Metric_Pad1.18x1.45mm_HandSolder, F.Cu at (238.5, 46.1)
- added C18: 470n, Capacitor_SMD:C_0805_2012Metric_Pad1.18x1.45mm_HandSolder, F.Cu at (238.5, 49.1)
- added C19: 470n, Capacitor_SMD:C_0805_2012Metric_Pad1.18x1.45mm_HandSolder, F.Cu at (238.5, 52.1)
- added C2: 100n, Capacitor_SMD:C_1206_3216Metric_Pad1.33x1.80mm_HandSolder, F.Cu at (116.6, 103.0)
- added C20: 470n, Capacitor_SMD:C_0805_2012Metric_Pad1.18x1.45mm_HandSolder, F.Cu at (238.5, 55.1)
- added C21: 470n, Capacitor_SMD:C_0805_2012Metric_Pad1.18x1.45mm_HandSolder, F.Cu at (238.5, 58.1)
- added C22: 470n, Capacitor_SMD:C_0805_2012Metric_Pad1.18x1.45mm_HandSolder, F.Cu at (243.3, 46.1)
- added C23: 330n, Capacitor_SMD:C_0805_2012Metric_Pad1.18x1.45mm_HandSolder, F.Cu at (243.3, 49.1)
- added C24: 330n, Capacitor_SMD:C_0805_2012Metric_Pad1.18x1.45mm_HandSolder, F.Cu at (243.3, 52.1)
- added C25: 10u, Capacitor_SMD:C_0805_2012Metric_Pad1.18x1.45mm_HandSolder, F.Cu at (243.3, 55.1)
- added C26: 10u, Capacitor_SMD:C_0805_2012Metric_Pad1.18x1.45mm_HandSolder, F.Cu at (243.3, 58.1)
- added C27: 2u2, Capacitor_SMD:C_0805_2012Metric_Pad1.18x1.45mm_HandSolder, F.Cu at (180.6, 123.2)
- added C28: 2u2, Capacitor_SMD:C_0805_2012Metric_Pad1.18x1.45mm_HandSolder, F.Cu at (189.3, 123.2)
- added C29: 10n, Capacitor_SMD:C_0805_2012Metric_Pad1.18x1.45mm_HandSolder, F.Cu at (176.2, 123.2)
- added C3: 100n, Capacitor_SMD:C_1206_3216Metric_Pad1.33x1.80mm_HandSolder, F.Cu at (133.8, 112.4)
- added C30: 10n, Capacitor_SMD:C_0805_2012Metric_Pad1.18x1.45mm_HandSolder, F.Cu at (184.9, 123.2)
- added C31: 10u, Capacitor_SMD:C_0805_2012Metric_Pad1.18x1.45mm_HandSolder, F.Cu at (178.4, 123.2)
- added C32: 10u, Capacitor_SMD:C_0805_2012Metric_Pad1.18x1.45mm_HandSolder, F.Cu at (187.1, 123.2)
- added C33: 2u2, Capacitor_SMD:C_0805_2012Metric_Pad1.18x1.45mm_HandSolder, F.Cu at (197.5, 123.2)
- added C34: 2u2, Capacitor_SMD:C_0805_2012Metric_Pad1.18x1.45mm_HandSolder, F.Cu at (238.6, 78.2)
- added C35: 10n, Capacitor_SMD:C_0805_2012Metric_Pad1.18x1.45mm_HandSolder, F.Cu at (193.3, 123.2)
- added C36: 10n, Capacitor_SMD:C_0805_2012Metric_Pad1.18x1.45mm_HandSolder, F.Cu at (244.0, 89.8)
- added C37: 10u, Capacitor_SMD:C_0805_2012Metric_Pad1.18x1.45mm_HandSolder, F.Cu at (195.4, 123.2)
- added C38: 10u, Capacitor_SMD:C_0805_2012Metric_Pad1.18x1.45mm_HandSolder, F.Cu at (238.6, 84.2)
- added C4: 100n, Capacitor_SMD:C_1206_3216Metric_Pad1.33x1.80mm_HandSolder, F.Cu at (133.8, 109.6)
- added C5: 10u, Capacitor_SMD:C_0805_2012Metric_Pad1.18x1.45mm_HandSolder, F.Cu at (131.6, 143.4)
- added C6: 22u, Capacitor_SMD:C_0805_2012Metric_Pad1.18x1.45mm_HandSolder, F.Cu at (138.8, 142.4)
- added C7: 22u, Capacitor_SMD:C_0805_2012Metric_Pad1.18x1.45mm_HandSolder, F.Cu at (138.8, 144.6)
- added C8: 22u, Capacitor_SMD:C_0805_2012Metric_Pad1.18x1.45mm_HandSolder, F.Cu at (138.8, 146.8)
- added C9: 10u, Capacitor_SMD:C_0805_2012Metric_Pad1.18x1.45mm_HandSolder, F.Cu at (120.4, 143.4)
- added D1: RED, LED_SMD:LED_0805_2012Metric, F.Cu at (151.8, 165.4)
- added D2: GREEN, LED_SMD:LED_0805_2012Metric, F.Cu at (151.7, 168.6)
- added D3: 5V Zener, Diode_THT:D_A-405_P7.62mm_Horizontal, F.Cu at (122.2, 147.4)
- added D4: RED, LED_SMD:LED_0805_2012Metric, F.Cu at (116.6, 133.2)
- added D5: SS14, Diode_SMD:D_SOD-123, F.Cu at (244.9, 30.2)
- added D6: SS14, Diode_SMD:D_SOD-123, F.Cu at (254.3, 34.8)
- added J1: CONN_MOTOR_1, Connector_JST:JST_EH_S2B-EH_1x02_P2.50mm_Horizontal, F.Cu at (178.6, 142.8)
- added J10: CONN_JTAG, Connector_PinHeader_2.54mm:PinHeader_1x06_P2.54mm_Vertical, F.Cu at (207.6, 123.9)
- added J11: CONN_FDBK_2, Connector_JST:JST_EH_S2B-EH_1x02_P2.50mm_Horizontal, F.Cu at (165.8, 142.7)
- added J12: CONN_EMG_2, Connector_JST:JST_EH_S3B-EH_1x03_P2.50mm_Horizontal, F.Cu at (157.2, 107.4)
- added J13: CONN_POS_3, Connector_JST:JST_EH_S3B-EH_1x03_P2.50mm_Horizontal, F.Cu at (170.8, 107.6)
- added J2: CONN_MOTOR_2, Connector_JST:JST_EH_S2B-EH_1x02_P2.50mm_Horizontal, F.Cu at (187.4, 142.8)
- added J3: CONN_BATT, Connector_JST:JST_EH_S2B-EH_1x02_P2.50mm_Horizontal, F.Cu at (107.1, 138.1)
- added J4: USB_C_CONN, Connector_USB:USB_C_Receptacle_G-Switch_GT-USB-7010ASV, F.Cu at (104.2, 114.4)
- added J5: CONN_POS_1, Connector_JST:JST_EH_S3B-EH_1x03_P2.50mm_Horizontal, F.Cu at (193.2, 107.6)
- added J6: CONN_MOTOR_3, Connector_JST:JST_EH_S2B-EH_1x02_P2.50mm_Horizontal, F.Cu at (196.2, 142.8)
- added J7: CONN_FDBK_1, Connector_JST:JST_EH_S2B-EH_1x02_P2.50mm_Horizontal, F.Cu at (156.6, 142.7)
- added J8: CONN_EMG_1, Connector_JST:JST_EH_S3B-EH_1x03_P2.50mm_Horizontal, F.Cu at (146.1, 107.4)
- added J9: CONN_POS_2, Connector_JST:JST_EH_S3B-EH_1x03_P2.50mm_Horizontal, F.Cu at (182.0, 107.6)
- added JP1: SolderJumper_2_Open, Jumper:SolderJumper-2_P1.3mm_Open_RoundedPad1.0x1.5mm, F.Cu at (123.7, 166.8)
- added JP10: JMPR_REVP, Jumper:SolderJumper-2_P1.3mm_Bridged_RoundedPad1.0x1.5mm, F.Cu at (119.0, 140.0)
- added JP11: JMPR_RST, Jumper:SolderJumper-2_P1.3mm_Bridged_RoundedPad1.0x1.5mm, F.Cu at (153.3, 66.8)
- added JP12: JMPR_BOOT, Jumper:SolderJumper-2_P1.3mm_Bridged_RoundedPad1.0x1.5mm, F.Cu at (153.3, 70.4)
- added JP13: JMPR_RX, Jumper:SolderJumper-2_P1.3mm_Bridged_RoundedPad1.0x1.5mm, F.Cu at (153.3, 74.0)
- added JP14: JMPR_TX, Jumper:SolderJumper-2_P1.3mm_Bridged_RoundedPad1.0x1.5mm, F.Cu at (153.3, 77.5)
- added JP15: JMPR_USB_N, Jumper:SolderJumper-2_P1.3mm_Bridged_RoundedPad1.0x1.5mm, F.Cu at (153.3, 81.0)
- added JP16: JMPR_USB_P, Jumper:SolderJumper-2_P1.3mm_Bridged_RoundedPad1.0x1.5mm, F.Cu at (157.7, 66.8)
- added JP17: JMPR_TRIM_1, Jumper:SolderJumper-2_P1.3mm_Bridged_RoundedPad1.0x1.5mm, F.Cu at (157.7, 70.4)
- added JP18: JMPR_TRIM_2, Jumper:SolderJumper-2_P1.3mm_Bridged_RoundedPad1.0x1.5mm, F.Cu at (157.7, 74.0)
- added JP19: JMPR_POT_1, Jumper:SolderJumper-2_P1.3mm_Bridged_RoundedPad1.0x1.5mm, F.Cu at (157.7, 77.5)
- added JP2: SolderJumper_2_Open, Jumper:SolderJumper-2_P1.3mm_Open_RoundedPad1.0x1.5mm, F.Cu at (123.7, 170.3)
- added JP20: JMPR_LED_1, Jumper:SolderJumper-2_P1.3mm_Bridged_RoundedPad1.0x1.5mm, F.Cu at (157.7, 81.0)
- added JP21: JMPR_LED_2, Jumper:SolderJumper-2_P1.3mm_Bridged_RoundedPad1.0x1.5mm, F.Cu at (162.0, 66.8)
- added JP22: JMPR_BTN_1, Jumper:SolderJumper-2_P1.3mm_Bridged_RoundedPad1.0x1.5mm, F.Cu at (162.0, 70.4)
- added JP23: JMPR_BTN_RST, Jumper:SolderJumper-2_P1.3mm_Bridged_RoundedPad1.0x1.5mm, F.Cu at (162.0, 74.0)
- added JP24: JMPR_BTN_BOOT, Jumper:SolderJumper-2_P1.3mm_Bridged_RoundedPad1.0x1.5mm, F.Cu at (162.0, 77.5)
- added JP3: SolderJumper_2_Open, Jumper:SolderJumper-2_P1.3mm_Open_RoundedPad1.0x1.5mm, F.Cu at (123.7, 173.4)
- added JP4: SolderJumper_2_Open, Jumper:SolderJumper-2_P1.3mm_Open_RoundedPad1.0x1.5mm, F.Cu at (123.7, 177.4)
- added JP5: SolderJumper_2_Open, Jumper:SolderJumper-2_P1.3mm_Open_RoundedPad1.0x1.5mm, F.Cu at (123.8, 163.2)
- added JP6: SolderJumper_2_Open, Jumper:SolderJumper-2_P1.3mm_Open_RoundedPad1.0x1.5mm, F.Cu at (128.0, 166.8)
- added JP7: SolderJumper_2_Open, Jumper:SolderJumper-2_P1.3mm_Open_RoundedPad1.0x1.5mm, F.Cu at (128.0, 170.3)
- added JP8: SolderJumper_2_Open, Jumper:SolderJumper-2_P1.3mm_Open_RoundedPad1.0x1.5mm, F.Cu at (128.0, 173.9)
- added JP9: JMPR_PSU, Jumper:SolderJumper-2_P1.3mm_Bridged_RoundedPad1.0x1.5mm, F.Cu at (133.4, 139.8)
- added L1: 1.5uH, Inductor_THT:L_Radial_D6.0mm_P4.00mm, F.Cu at (125.8, 138.0)
- added Q1: 2N7002, Package_TO_SOT_SMD:SOT-23, F.Cu at (126.6, 114.0)
- added Q2: 2N7002, Package_TO_SOT_SMD:SOT-23, F.Cu at (126.6, 110.2)
- added Q3: PMOS, Package_DIP:Vishay_HVM-DIP-3_W7.62mm, F.Cu at (115.3, 136.6)
- added R1: 5k1, Resistor_SMD:R_0805_2012Metric_Pad1.20x1.40mm_HandSolder, F.Cu at (110.4, 104.0)
- added R10: 10k, Resistor_SMD:R_0805_2012Metric_Pad1.20x1.40mm_HandSolder, F.Cu at (185.4, 34.2)
- added R11: 4k7, Resistor_SMD:R_0805_2012Metric_Pad1.20x1.40mm_HandSolder, F.Cu at (185.4, 37.2)
- added R12: 10k, Resistor_SMD:R_0805_2012Metric_Pad1.20x1.40mm_HandSolder, F.Cu at (122.6, 143.4)
- added R13: 680k, Resistor_SMD:R_0805_2012Metric_Pad1.20x1.40mm_HandSolder, F.Cu at (134.8, 142.4)
- added R14: 100k, Resistor_SMD:R_0805_2012Metric_Pad1.20x1.40mm_HandSolder, F.Cu at (131.4, 146.8)
- added R15: 47k, Resistor_SMD:R_0805_2012Metric_Pad1.20x1.40mm_HandSolder, F.Cu at (112.2, 147.4)
- added R16: 130k, Resistor_SMD:R_0805_2012Metric_Pad1.20x1.40mm_HandSolder, F.Cu at (134.8, 144.6)
- added R17: 4k7, Resistor_SMD:R_0805_2012Metric_Pad1.20x1.40mm_HandSolder, F.Cu at (113.4, 134.0)
- added R18: 47k, Resistor_SMD:R_0805_2012Metric_Pad1.20x1.40mm_HandSolder, F.Cu at (217.5, 25.4)
- added R19: 47k, Resistor_SMD:R_0805_2012Metric_Pad1.20x1.40mm_HandSolder, F.Cu at (217.5, 28.4)
- added R2: 5k1, Resistor_SMD:R_0805_2012Metric_Pad1.20x1.40mm_HandSolder, F.Cu at (112.6, 104.0)
- added R20: 15k, Resistor_SMD:R_0805_2012Metric_Pad1.20x1.40mm_HandSolder, F.Cu at (217.5, 31.3)
- added R21: 15k, Resistor_SMD:R_0805_2012Metric_Pad1.20x1.40mm_HandSolder, F.Cu at (217.5, 34.2)
- added R22: 1k, Resistor_SMD:R_0805_2012Metric_Pad1.20x1.40mm_HandSolder, F.Cu at (217.5, 37.2)
- added R23: 1k, Resistor_SMD:R_0805_2012Metric_Pad1.20x1.40mm_HandSolder, F.Cu at (217.5, 40.1)
- added R24: 1k, Resistor_SMD:R_0805_2012Metric_Pad1.20x1.40mm_HandSolder, F.Cu at (217.5, 43.1)
- added R25: 1k, Resistor_SMD:R_0805_2012Metric_Pad1.20x1.40mm_HandSolder, F.Cu at (222.3, 25.4)
- added R26: 1k, Resistor_SMD:R_0805_2012Metric_Pad1.20x1.40mm_HandSolder, F.Cu at (222.3, 28.4)
- added R27: 1k, Resistor_SMD:R_0805_2012Metric_Pad1.20x1.40mm_HandSolder, F.Cu at (222.3, 31.3)
- added R28: 47k, Resistor_SMD:R_0805_2012Metric_Pad1.20x1.40mm_HandSolder, F.Cu at (222.3, 34.2)
- added R29: 15k, Resistor_SMD:R_0805_2012Metric_Pad1.20x1.40mm_HandSolder, F.Cu at (222.3, 37.2)
- added R3: 1k, Resistor_SMD:R_0805_2012Metric_Pad1.20x1.40mm_HandSolder, F.Cu at (123.3, 114.4)
- added R30: 47k, Resistor_SMD:R_0805_2012Metric_Pad1.20x1.40mm_HandSolder, F.Cu at (222.3, 40.1)
- added R31: 15k, Resistor_SMD:R_0805_2012Metric_Pad1.20x1.40mm_HandSolder, F.Cu at (222.3, 43.1)
- added R32: 10k, Resistor_SMD:R_0805_2012Metric_Pad1.20x1.40mm_HandSolder, F.Cu at (227.0, 25.4)
- added R33: 10k, Resistor_SMD:R_0805_2012Metric_Pad1.20x1.40mm_HandSolder, F.Cu at (227.0, 28.4)
- added R34: 18k, Resistor_SMD:R_0805_2012Metric_Pad1.20x1.40mm_HandSolder, F.Cu at (227.0, 31.3)
- added R35: 18k, Resistor_SMD:R_0805_2012Metric_Pad1.20x1.40mm_HandSolder, F.Cu at (227.0, 34.2)
- added R36: 1k, Resistor_SMD:R_0805_2012Metric_Pad1.20x1.40mm_HandSolder, F.Cu at (227.0, 37.2)
- added R37: 1k, Resistor_SMD:R_0805_2012Metric_Pad1.20x1.40mm_HandSolder, F.Cu at (227.0, 40.1)
- added R38: 47k, Resistor_SMD:R_0805_2012Metric_Pad1.20x1.40mm_HandSolder, F.Cu at (227.0, 43.1)
- added R39: 47k, Resistor_SMD:R_0805_2012Metric_Pad1.20x1.40mm_HandSolder, F.Cu at (231.8, 25.4)
- added R4: 1k, Resistor_SMD:R_0805_2012Metric_Pad1.20x1.40mm_HandSolder, F.Cu at (123.3, 110.4)
- added R40: 1k, Resistor_SMD:R_0805_2012Metric_Pad1.20x1.40mm_HandSolder, F.Cu at (231.8, 28.4)
- added R41: 1k, Resistor_SMD:R_0805_2012Metric_Pad1.20x1.40mm_HandSolder, F.Cu at (231.8, 31.3)
- added R42: 10k, Resistor_SMD:R_0805_2012Metric_Pad1.20x1.40mm_HandSolder, F.Cu at (231.8, 34.2)
- added R43: 10k, Resistor_SMD:R_0805_2012Metric_Pad1.20x1.40mm_HandSolder, F.Cu at (231.8, 37.2)
- added R44: 18k, Resistor_SMD:R_0805_2012Metric_Pad1.20x1.40mm_HandSolder, F.Cu at (231.8, 40.1)
- added R45: 18k, Resistor_SMD:R_0805_2012Metric_Pad1.20x1.40mm_HandSolder, F.Cu at (231.8, 43.1)
- added R46: 18k, Resistor_SMD:R_0805_2012Metric_Pad1.20x1.40mm_HandSolder, F.Cu at (236.5, 25.4)
- added R47: 18k, Resistor_SMD:R_0805_2012Metric_Pad1.20x1.40mm_HandSolder, F.Cu at (236.5, 28.4)
- added R48: 10k, Resistor_SMD:R_0805_2012Metric_Pad1.20x1.40mm_HandSolder, F.Cu at (236.5, 31.3)
- added R49: 10k, Resistor_SMD:R_0805_2012Metric_Pad1.20x1.40mm_HandSolder, F.Cu at (236.5, 34.2)
- added R5: 10k, Resistor_SMD:R_0805_2012Metric_Pad1.20x1.40mm_HandSolder, F.Cu at (180.7, 37.2)
- added R50: 10k, Resistor_SMD:R_0805_2012Metric_Pad1.20x1.40mm_HandSolder, F.Cu at (236.5, 37.2)
- added R51: 47k, Resistor_SMD:R_0805_2012Metric_Pad1.20x1.40mm_HandSolder, F.Cu at (236.5, 40.1)
- added R52: 10k, Resistor_SMD:R_0805_2012Metric_Pad1.20x1.40mm_HandSolder, F.Cu at (236.5, 43.1)
- added R53: 0R200, Resistor_SMD:R_1206_3216Metric_Pad1.30x1.75mm_HandSolder, F.Cu at (177.1, 134.6)
- added R54: 0R200, Resistor_SMD:R_1206_3216Metric_Pad1.30x1.75mm_HandSolder, F.Cu at (185.5, 134.8)
- added R55: 4R7, Resistor_SMD:R_1206_3216Metric_Pad1.30x1.75mm_HandSolder, F.Cu at (244.0, 69.8)
- added R56: 0R200, Resistor_SMD:R_1206_3216Metric_Pad1.30x1.75mm_HandSolder, F.Cu at (193.7, 134.8)
- added R57: 4R7, Resistor_SMD:R_1206_3216Metric_Pad1.30x1.75mm_HandSolder, F.Cu at (244.0, 76.4)
- added R6: 10k, Resistor_SMD:R_0805_2012Metric_Pad1.20x1.40mm_HandSolder, F.Cu at (180.7, 40.1)
- added R7: 10k, Resistor_SMD:R_0805_2012Metric_Pad1.20x1.40mm_HandSolder, F.Cu at (185.4, 25.4)
- added R8: 10k, Resistor_SMD:R_0805_2012Metric_Pad1.20x1.40mm_HandSolder, F.Cu at (185.4, 28.4)
- added R9: 4k7, Resistor_SMD:R_0805_2012Metric_Pad1.20x1.40mm_HandSolder, F.Cu at (185.4, 31.3)
- added RV1: TRIM_POT_1, Potentiometer_SMD:Potentiometer_Vishay_TS53YJ_Vertical, F.Cu at (202.4, 129.0)
- added RV2: TRIM_POT_2, Potentiometer_SMD:Potentiometer_Vishay_TS53YJ_Vertical, F.Cu at (202.4, 135.2)
- added RV3: POT_1, Potentiometer_SMD:Potentiometer_Vishay_TS53YJ_Vertical, F.Cu at (146.0, 143.2)
- added RV4: 100k, Potentiometer_SMD:Potentiometer_Vishay_TS53YJ_Vertical, F.Cu at (159.2, 128.0)
- added RV5: 100k, Potentiometer_SMD:Potentiometer_Vishay_TS53YJ_Vertical, F.Cu at (149.0, 128.2)
- added SW1: SW_Push, Button_Switch_SMD:SW_Tactile_SPST_NO_Straight_CK_PTS636Sx25SMTRLFS, F.Cu at (201.5, 120.8)
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Other:
- board size 110 x 40 mm -> 110 x 50 mm
- copper layers 2 -> 4
- board text added: "+ 1 -"
- board text added: "+ 2 -"
- board text added: "+ 3 -"
- board text added: "+ BATT -"
- board text added: "BOOT"
- board text added: "BTN"
- board text added: "HAPTIC FDBK"
- board text added: "JTAG"
- board text added: "MOTORS"
- board text added: "POT_1"
- board text added: "RST"
- board text added: "TRIM_1"
- board text added: "TRIM_2"
- board text added: "USB TYPE C"
- board text removed: "Board size: 40x110mm"

Commit message: Update schm and pcb
Parts:
- removed the R23 at (217.5, 40.1)
- removed the R30 at (222.3, 40.1)
- removed the R37 at (227.0, 40.1)
- removed the R44 at (231.8, 40.1)
- removed the R51 at (236.5, 40.1)
- removed TP1: TP_UC_RST, TestPoint:TestPoint_Pad_D1.0mm
- removed TP17: TP_BATT_P, TestPoint:TestPoint_Pad_D1.0mm
- removed TP18: TP_V_BATT, TestPoint:TestPoint_Pad_D1.0mm
- removed TP19: TP_V_5V, TestPoint:TestPoint_Pad_D1.0mm
- removed TP2: TP_UC_RX, TestPoint:TestPoint_Pad_D1.0mm
- removed TP20: TP_PSU_FDBK, TestPoint:TestPoint_Pad_D1.0mm
- removed TP21: TP_V_3V3, TestPoint:TestPoint_Pad_D1.0mm
- removed TP22: TP_V_N5V, TestPoint:TestPoint_Pad_D1.0mm
- removed TP28: TP_MOT_2_EN, TestPoint:TestPoint_Pad_D1.0mm
- removed TP29: TP_MOT_1_EN, TestPoint:TestPoint_Pad_D1.0mm
- removed TP3: TP_UC_TX, TestPoint:TestPoint_Pad_D1.0mm
- removed TP30: TP_MOT_1_FAULT, TestPoint:TestPoint_Pad_D1.0mm
- removed TP31: TP_MOT_2_FAULT, TestPoint:TestPoint_Pad_D1.0mm
- removed TP32: TP_MOT_1_IS, TestPoint:TestPoint_Pad_D1.0mm
- removed TP33: TP_MOT_2_IS, TestPoint:TestPoint_Pad_D1.0mm
- removed TP34: TP_MOT_2_UC1, TestPoint:TestPoint_Pad_D1.0mm
- removed TP35: TP_MOT_1_UC1, TestPoint:TestPoint_Pad_D1.0mm
- removed TP36: TP_MOT_1_OUT_P, TestPoint:TestPoint_Pad_D1.0mm
- removed TP37: TP_MOT_2_OUT_P, TestPoint:TestPoint_Pad_D1.0mm
- removed TP38: TP_MOT_1_UC2, TestPoint:TestPoint_Pad_D1.0mm
- removed TP39: TP_MOT_2_UC2, TestPoint:TestPoint_Pad_D1.0mm
- removed TP4: TP_USB_D_P, TestPoint:TestPoint_Pad_D1.0mm
- removed TP40: TP_MOT_1_OUT_N, TestPoint:TestPoint_Pad_D1.0mm
- removed TP41: TP_MOT_2_OUT_N, TestPoint:TestPoint_Pad_D1.0mm
- removed TP42: TP_MOT_3_EN, TestPoint:TestPoint_Pad_D1.0mm
- removed TP44: TP_MOT_3_FAULT, TestPoint:TestPoint_Pad_D1.0mm
- removed TP47: TP_MOT_3_IS, TestPoint:TestPoint_Pad_D1.0mm
- removed TP48: TP_MOT_3_UC1, TestPoint:TestPoint_Pad_D1.0mm
- removed TP5: TP_USB_D_N, TestPoint:TestPoint_Pad_D1.0mm
- removed TP50: TP_MOT_3_OUT_P, TestPoint:TestPoint_Pad_D1.0mm
- removed TP51: TP_MOT_3_UC2, TestPoint:TestPoint_Pad_D1.0mm
- removed TP52: TP_MOT_3_OUT_N, TestPoint:TestPoint_Pad_D1.0mm
- removed TP6: TP_UC_BOOT, TestPoint:TestPoint_Pad_D1.0mm
- added JP23: JMPR_REVP, Jumper:SolderJumper-2_P1.3mm_Bridged_RoundedPad1.0x1.5mm, F.Cu at (101.4, 29.0)
- added JP24: JMPR_PSU, Jumper:SolderJumper-2_P1.3mm_Bridged_RoundedPad1.0x1.5mm, F.Cu at (101.4, 32.5)
- added JP25: JMPR_EMG_2_UC, Jumper:SolderJumper-2_P1.3mm_Bridged_RoundedPad1.0x1.5mm, F.Cu at (100.8, 39.6)
- added JP26: JMPR_EMG_1_UC, Jumper:SolderJumper-2_P1.3mm_Bridged_RoundedPad1.0x1.5mm, F.Cu at (100.8, 36.1)
- added JP27: JMPR_I2C_ADC_SCL, Jumper:SolderJumper-2_P1.3mm_Bridged_RoundedPad1.0x1.5mm, F.Cu at (198.9, 121.7)
- added JP28: JMPR_I2C_ADC_SDA, Jumper:SolderJumper-2_P1.3mm_Bridged_RoundedPad1.0x1.5mm, F.Cu at (195.1, 121.7)
- added JP31: JMPR_MOT_1_EN, Jumper:SolderJumper-2_P1.3mm_Bridged_RoundedPad1.0x1.5mm, F.Cu at (105.5, 29.3)
- added JP32: JMPR_MOT_2_EN, Jumper:SolderJumper-2_P1.3mm_Bridged_RoundedPad1.0x1.5mm, F.Cu at (105.5, 32.9)
- added JP33: JMPR_MOT_1_UC1, Jumper:SolderJumper-2_P1.3mm_Bridged_RoundedPad1.0x1.5mm, F.Cu at (105.5, 36.4)
- added JP34: JMPR_MOT_2_UC1, Jumper:SolderJumper-2_P1.3mm_Bridged_RoundedPad1.0x1.5mm, F.Cu at (109.8, 29.3)
- added JP35: JMPR_MOT_1_UC2, Jumper:SolderJumper-2_P1.3mm_Bridged_RoundedPad1.0x1.5mm, F.Cu at (109.8, 32.9)
- added JP36: JMPR_MOT_2_UC2, Jumper:SolderJumper-2_P1.3mm_Bridged_RoundedPad1.0x1.5mm, F.Cu at (109.8, 36.4)
- added JP37: JMPR_MOT_3_EN, Jumper:SolderJumper-2_P1.3mm_Bridged_RoundedPad1.0x1.5mm, F.Cu at (114.2, 29.3)
- added JP38: JMPR_MOT_3_UC1, Jumper:SolderJumper-2_P1.3mm_Bridged_RoundedPad1.0x1.5mm, F.Cu at (114.2, 32.9)
- added JP39: JMPR_MOT_3_UC2, Jumper:SolderJumper-2_P1.3mm_Bridged_RoundedPad1.0x1.5mm, F.Cu at (114.2, 36.4)
- added R12: 10k, Resistor_SMD:R_0805_2012Metric_Pad1.20x1.40mm_HandSolder, F.Cu at (253.1, 42.5)
- added R13: 10k, Resistor_SMD:R_0805_2012Metric_Pad1.20x1.40mm_HandSolder, F.Cu at (253.1, 45.5)
- added R14: 10k, Resistor_SMD:R_0805_2012Metric_Pad1.20x1.40mm_HandSolder, F.Cu at (253.1, 36.6)
- added R15: 10k, Resistor_SMD:R_0805_2012Metric_Pad1.20x1.40mm_HandSolder, F.Cu at (253.1, 39.5)
- added R27: 1k, Resistor_SMD:R_0805_2012Metric_Pad1.20x1.40mm_HandSolder, F.Cu at (232.4, 47.1)
- added R34: 47k, Resistor_SMD:R_0805_2012Metric_Pad1.20x1.40mm_HandSolder, F.Cu at (232.4, 50.0)
- added R41: 1k, Resistor_SMD:R_0805_2012Metric_Pad1.20x1.40mm_HandSolder, F.Cu at (232.4, 53.0)
- added R50: 18k, Resistor_SMD:R_0805_2012Metric_Pad1.20x1.40mm_HandSolder, F.Cu at (232.4, 56.0)
- added R52: 10k, Resistor_SMD:R_0805_2012Metric_Pad1.20x1.40mm_HandSolder, F.Cu at (207.9, 119.2)
- added R54: 47k, Resistor_SMD:R_0805_2012Metric_Pad1.20x1.40mm_HandSolder, F.Cu at (132.5, 148.6)
- added R56: 10k, Resistor_SMD:R_1206_3216Metric_Pad1.30x1.75mm_HandSolder, F.Cu at (245.2, 39.5)
- added R57: 10k, Resistor_SMD:R_1206_3216Metric_Pad1.30x1.75mm_HandSolder, F.Cu at (245.2, 42.8)
- added R60: 10k, Resistor_SMD:R_1206_3216Metric_Pad1.30x1.75mm_HandSolder, F.Cu at (245.2, 36.2)
- added R61: 10k, Resistor_SMD:R_1206_3216Metric_Pad1.30x1.75mm_HandSolder, F.Cu at (245.2, 46.1)
- added U8: ADS1115IDGS, Package_SO:TSSOP-10_3x3mm_P0.5mm, F.Cu at (205.0, 119.2)
- R58: renamed from R53; value 0R200 -> 0R2
- R59: renamed from R54; value 0R200 -> 0R2
- R63: renamed from R56; value 0R200 -> 0R2
- RV1: renamed from RV3; value POT_1 -> TRIM_POT_3
- moved R7 147.6 mm to (54.9, 94.2)
- moved R55 145.4 mm to (136.5, 148.6), turned to 180 degrees
- moved R5 141.5 mm to (47.9, 86.0)
- moved R6 141.5 mm to (47.9, 89.0)
- moved JP13 123.9 mm to (29.4, 97.0)
- moved JP10 120.7 mm to (33.2, 87.0)
- moved JP12 120.7 mm to (33.2, 93.5)
- moved JP16 120.7 mm to (37.5, 87.0)
- moved JP18 120.7 mm to (37.5, 94.0)
- moved JP11 120.7 mm to (33.2, 90.5)
- moved JP15 120.7 mm to (33.3, 83.3)
- moved JP17 120.7 mm to (37.5, 90.5)
- moved R9 97.4 mm to (131.3, 112.3), turned to 180 degrees
- moved R11 94.3 mm to (131.3, 114.4), turned to 180 degrees
- moved JP10 90.0 mm to (41.5, 94.4)
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- renumbered C26 to C25, C25 to C26, JP11 to JP1, JP1 to JP10, JP2 to JP11, JP3 to JP12, JP4 to JP13, JP20 to JP14, JP5 to JP15, JP6 to JP16, JP7 to JP17, JP8 to JP18, JP22 to JP19, JP13 to JP2, JP21 to JP20, JP23 to JP21, JP24 to JP22, JP14 to JP3, JP16 to JP4, JP15 to JP5, JP12 to JP6, JP19 to JP7, JP17 to JP8, JP18 to JP9, R12 to R16, R13 to R17, R14 to R18, R15 to R19, R16 to R20, R17 to R21, R18 to R22, R19 to R23, R20 to R24, R21 to R25, R22 to R26, R24 to R28, R26 to R29, R25 to R30, R27 to R31, R28 to R32, R29 to R33, R31 to R35, R32 to R36, R33 to R37, R34 to R38, R35 to R39, R36 to R40, R38 to R42, R40 to R43, R39 to R44, R41 to R45, R42 to R46, R43 to R47, R45 to R48, R46 to R49, R47 to R51, R48 to R53, R52 to R55, R55 to R62, R57 to R64, RV1 to RV2, RV2 to RV3, U9 to U10, U10 to U11, U11 to U12, U12 to U13, U8 to U9
Connections:
- net BAT_N renamed Earth
- net EMG_1_UC renamed Net-(D6-K)
- net EMG_2_UC renamed Net-(D5-K)
- net MOTOR_1_UC1 renamed Net-(JP33-B)
- net MOTOR_1_UC2 renamed Net-(JP35-A)
- net MOTOR_2_UC1 renamed Net-(JP34-B)
- net MOTOR_2_UC2 renamed Net-(JP36-A)
- net MOTOR_3_UC1 renamed Net-(JP38-B)
- net MOTOR_3_UC2 renamed Net-(JP39-A)
- C5 pad 1: Net-(JP9-A) -> Net-(JP24-A)
- C6 pad 1: Net-(JP9-A) -> +5V
- C7 pad 1: Net-(JP9-A) -> +5V
- C8 pad 1: Net-(JP9-A) -> +5V
- JP19 pad 1: Net-(JP22-A) -> Net-(JP19-A)
- JP22 pad 1: Net-(JP24-A) -> Net-(JP22-A)
- JP7 pad 1: Net-(JP19-A) -> Net-(JP7-A)
- JP7 pad 2: POT_1 -> TRIM_POT_3
- JP8 pad 1: Net-(JP17-A) -> Net-(JP8-A)
- JP9 pad 1: Net-(JP18-A) -> Net-(JP9-A)
- R10 pad 2: Net-(JP22-A) -> Net-(JP19-A)
- R16 pad 2: +BATT -> Net-(JP23-B)
- R17 pad 2: Net-(JP9-A) -> Net-(JP24-A)
- R18 pad 2: Net-(JP9-A) -> Net-(JP24-A)
- R53 pad 1: ADC_ALERT_RDY -> ADC_1_ALERT_RDY
- R55 pad 2: Net-(U8-AIN0) -> Net-(U9-AIN0)
- RV1 pad 2: Net-(JP19-A) -> Net-(JP7-A)
- RV2 pad 2: Net-(JP17-A) -> Net-(JP8-A)
- RV3 pad 2: Net-(JP18-A) -> Net-(JP9-A)
- SW1 pad 1: Net-(JP22-A) -> Net-(JP19-A)
- SW3 pad 1: Net-(JP24-A) -> Net-(JP22-A)
- U10 pad 1: MOTOR_1_EN -> Net-(JP31-B)
- U11 pad 1: MOTOR_2_EN -> Net-(JP32-B)
- U12 pad 1: MOTOR_3_EN -> Net-(JP37-B)
- U3 pad 12: +BATT -> Net-(JP23-B)
- U3 pad 13: +BATT -> Net-(JP23-B)
- U3 pad 7: Net-(JP9-A) -> Net-(JP24-A)
- U3 pad 8: Net-(JP9-A) -> Net-(JP24-A)
- U9 pad 10: UC_SCL -> ADC_SCL
- U9 pad 2: ADC_ALERT_RDY -> ADC_1_ALERT_RDY
- U9 pad 4: Net-(U8-AIN0) -> Net-(U9-AIN0)
- U9 pad 9: UC_SDA -> ADC_SDA
Other:
- board text added: "+ -"
- board text added: "-"
- board text added: "1"
- board text added: "2"
- board text added: "BAT"
- board text added: "EMG"
- board text added: "HAPTIC"
- board text added: "POS"
- board text added: "POTS"
- board text added: "USB C"
- board text removed: "+ BATT -"
- board text removed: "HAPTIC FDBK"
- board text removed: "POT_1"
- board text removed: "TRIM_1"
- board text removed: "TRIM_2"
- board text removed: "USB TYPE C"

Commit message: Update schm and pcb
Parts:
- removed the JP10 at (33.2, 87.0)
- removed the JP10 at (41.5, 94.4)
- removed the R5 at (47.9, 86.0)
- removed the R6 at (47.9, 89.0)
- removed TP9: TP_POT_1, TestPoint:TestPoint_Pad_D1.0mm
- added JP10: SolderJumper_2_Open, Jumper:SolderJumper-2_P1.3mm_Open_RoundedPad1.0x1.5mm, F.Cu at (45.1, 110.9)
- added R10: 10k, Resistor_SMD:R_0805_2012Metric_Pad1.20x1.40mm_HandSolder, F.Cu at (54.0, 119.5)
- added R9: 10k, Resistor_SMD:R_0805_2012Metric_Pad1.20x1.40mm_HandSolder, F.Cu at (54.0, 116.5)
- added TP1: TP_UC_RST, TestPoint:TestPoint_Pad_D1.0mm, F.Cu at (55.8, 32.7)
- added TP17: TP_UC_PIN_PD1, TestPoint:TestPoint_Pad_D1.0mm, F.Cu at (61.9, 38.8)
- added TP18: TP_HW_REV_4, TestPoint:TestPoint_Pad_D1.0mm, F.Cu at (61.9, 41.9)
- added TP19: TP_UC_PIN_PD2, TestPoint:TestPoint_Pad_D1.0mm, F.Cu at (65.0, 32.7)
- added TP2: TP_USB_D_P, TestPoint:TestPoint_Pad_D1.0mm, F.Cu at (112.2, 115.7)
- added TP20: TP_UC_PIN_PC0, TestPoint:TestPoint_Pad_D1.0mm, F.Cu at (65.0, 35.8)
- added TP22: TP_UC_PIN_PC1, TestPoint:TestPoint_Pad_D1.0mm, F.Cu at (65.0, 38.8)
- added TP28: TP_UC_PIN_PB5, TestPoint:TestPoint_Pad_D1.0mm, F.Cu at (68.0, 41.9)
- added TP29: TP_UC_PIN_PC14, TestPoint:TestPoint_Pad_D1.0mm, F.Cu at (71.0, 32.7)
- added TP3: TP_USB_D_N, TestPoint:TestPoint_Pad_D1.0mm, F.Cu at (112.2, 107.9)
- added TP30: TP_UC_PIN_PC15, TestPoint:TestPoint_Pad_D1.0mm, F.Cu at (71.0, 35.8)
- added TP31: TP_UC_PIN_PB10, TestPoint:TestPoint_Pad_D1.0mm, F.Cu at (71.0, 38.8)
- added TP32: TP_UC_PIN_PB11, TestPoint:TestPoint_Pad_D1.0mm, F.Cu at (71.0, 41.9)
- added TP33: TP_BATT_P, TestPoint:TestPoint_Pad_D1.0mm, F.Cu at (109.9, 142.7)
- added TP34: TP_V_BATT, TestPoint:TestPoint_Pad_D1.0mm, F.Cu at (109.9, 145.1)
- added TP35: TP_V_5V, TestPoint:TestPoint_Pad_D1.0mm, F.Cu at (135.4, 139.9)
- added TP36: TP_PSU_FDBK, TestPoint:TestPoint_Pad_D1.0mm, F.Cu at (129.7, 140.5)
- added TP37: TP_V_3V3, TestPoint:TestPoint_Pad_D1.0mm, F.Cu at (102.0, 121.7)
- added TP38: TP_V_N5V, TestPoint:TestPoint_Pad_D1.0mm, F.Cu at (113.9, 121.7)
- added TP39: TP_EMG_2_AMP, TestPoint:TestPoint_Pad_D1.0mm, F.Cu at (55.8, 46.9)
- added TP4: TP_UC_BOOT, TestPoint:TestPoint_Pad_D1.0mm, F.Cu at (55.8, 35.8)
- added TP40: TP_EMG_1_AMP, TestPoint:TestPoint_Pad_D1.0mm, F.Cu at (55.8, 50.0)
- added TP41: TP_EMG_2_HP, TestPoint:TestPoint_Pad_D1.0mm, F.Cu at (55.8, 53.0)
- added TP42: TP_EMG_1_HP, TestPoint:TestPoint_Pad_D1.0mm, F.Cu at (58.9, 46.9)
- added TP44: TP_EMG_1_UC, TestPoint:TestPoint_Pad_D1.0mm, F.Cu at (58.9, 53.0)
- added TP47: TP_ADC_RDY, TestPoint:TestPoint_Pad_D1.0mm, F.Cu at (139.3, 131.9)
- added TP48: TP_TRIM_1, TestPoint:TestPoint_Pad_D1.0mm, F.Cu at (189.3, 112.3)
- added TP49: TP_TRIM_2, TestPoint:TestPoint_Pad_D1.0mm, F.Cu at (195.3, 112.3)
- added TP50: TP_TRIM_3, TestPoint:TestPoint_Pad_D1.0mm, F.Cu at (201.2, 112.2)
- added TP51: TP_TRIM_4, TestPoint:TestPoint_Pad_D1.0mm, F.Cu at (181.3, 124.8)
- added TP52: TP_ADC_RDY, TestPoint:TestPoint_Pad_D1.0mm, F.Cu at (61.9, 53.0)
- added TP55: TP_HALL_02, TestPoint:TestPoint_Pad_D1.0mm, F.Cu at (180.9, 112.3)
- added TP56: TP_HALL_03, TestPoint:TestPoint_Pad_D1.0mm, F.Cu at (178.7, 112.3)
- added TP57: TP_MOT_1_EN, TestPoint:TestPoint_Pad_D1.0mm, F.Cu at (41.6, 32.7)
- added TP58: TP_MOT_2_EN, TestPoint:TestPoint_Pad_D1.0mm, F.Cu at (41.6, 35.8)
- added TP59: TP_MOT_1_IS, TestPoint:TestPoint_Pad_D1.0mm, F.Cu at (41.6, 38.8)
- added TP60: TP_MOT_1_FAULT, TestPoint:TestPoint_Pad_D1.0mm, F.Cu at (41.6, 41.9)
- added TP61: TP_MOT_2_IS, TestPoint:TestPoint_Pad_D1.0mm, F.Cu at (41.6, 44.9)
- added TP62: TP_MOT_2_FAULT, TestPoint:TestPoint_Pad_D1.0mm, F.Cu at (41.6, 48.0)
- added TP63: TP_MOT_1_UC1, TestPoint:TestPoint_Pad_D1.0mm, F.Cu at (41.6, 51.0)
- added TP64: TP_MOT_2_UC1, TestPoint:TestPoint_Pad_D1.0mm, F.Cu at (44.6, 32.7)
- added TP65: TP_MOT_1_UC2, TestPoint:TestPoint_Pad_D1.0mm, F.Cu at (44.6, 35.8)
- added TP66: TP_MOT_2_UC2, TestPoint:TestPoint_Pad_D1.0mm, F.Cu at (44.6, 38.8)
- added TP67: TP_MOT_1_OUT_P, TestPoint:TestPoint_Pad_D1.0mm, F.Cu at (44.6, 41.9)
- added TP68: TP_MOT_2_OUT_P, TestPoint:TestPoint_Pad_D1.0mm, F.Cu at (44.6, 44.9)
- added TP69: TP_MOT_1_OUT_N, TestPoint:TestPoint_Pad_D1.0mm, F.Cu at (44.6, 48.0)
- added TP70: TP_MOT_2_OUT_N, TestPoint:TestPoint_Pad_D1.0mm, F.Cu at (44.6, 51.0)
- added TP71: TP_MOT_3_EN, TestPoint:TestPoint_Pad_D1.0mm, F.Cu at (47.7, 32.7)
- added TP72: TP_FDBK_MOT_EN, TestPoint:TestPoint_Pad_D1.0mm, F.Cu at (47.7, 35.8)
- added TP73: TP_MOT_3_IS, TestPoint:TestPoint_Pad_D1.0mm, F.Cu at (47.7, 38.8)
- added TP74: TP_MOT_3_FAULT, TestPoint:TestPoint_Pad_D1.0mm, F.Cu at (47.7, 41.9)
- added TP75: TP_FDBK_MOT_FAULT, TestPoint:TestPoint_Pad_D1.0mm, F.Cu at (47.7, 44.9)
- added TP76: TP_MOT_3_UC1, TestPoint:TestPoint_Pad_D1.0mm, F.Cu at (47.7, 48.0)
- added TP77: TP_FDBK_MOT_1_UC1, TestPoint:TestPoint_Pad_D1.0mm, F.Cu at (47.7, 51.0)
- added TP78: TP_MOT_3_UC2, TestPoint:TestPoint_Pad_D1.0mm, F.Cu at (50.8, 32.7)
- added TP79: TP_FDBK_MOT_1_UC2, TestPoint:TestPoint_Pad_D1.0mm, F.Cu at (50.8, 35.8)
- added TP80: TP_MOT_3_OUT_P, TestPoint:TestPoint_Pad_D1.0mm, F.Cu at (50.8, 38.8)
- added TP81: TP_MOT_3_OUT_N, TestPoint:TestPoint_Pad_D1.0mm, F.Cu at (50.8, 41.9)
- added TP82: TP_FDBK_MOT_2_UC1, TestPoint:TestPoint_Pad_D1.0mm, F.Cu at (50.8, 44.9)
- added TP83: TP_FDBK_MOT_2_UC2, TestPoint:TestPoint_Pad_D1.0mm, F.Cu at (50.8, 48.0)
- TP10: value TP_HW_REV_2 -> TP_HW_REV_1
- TP11: value TP_HW_REV_1 -> TP_HW_REV_2
- TP12: value TP_LED_1 -> TP_UC_PIN_PD0
- TP13: value TP_HW_REV_3 -> TP_UC_RX
- TP14: value TP_BTN_1 -> TP_LED_1
- TP15: value TP_LED_2 -> TP_UC_TX
- TP16: value TP_HW_REV_4 -> TP_HW_REV_3
- TP23: value TP_ADC_RDY -> TP_LED_2
- TP24: value TP_BATT_SENSE -> TP_UC_PIN_PC2
- TP25: value TP_HALL_01 -> TP_UC_PIN_PC3
- TP26: value TP_HALL_02 -> TP_UC_PIN_PB2
- TP27: value TP_HALL_03 -> TP_UC_PIN_PC13
- TP43: value TP_FDBK_MOT_EN -> TP_EMG_2_UC
- TP45: value TP_FDBK_MOT_1_UC2 -> TP_EMG_2_LP
- TP46: value TP_FDBK_MOT_FAULT -> TP_EMG_1_LP
- TP53: value TP_FDBK_MOT_2_UC1 -> TP_BATT_SENSE
- TP54: value TP_FDBK_MOT_2_UC2 -> TP_HALL_01
- TP7: value TP_TRIM_POT_1 -> TP_UC_SCL
- TP8: value TP_TRIM_POT_2 -> TP_UC_SDA
- moved R8 220.7 mm to (54.0, 113.5)
- moved R15 145.4 mm to (124.6, 107.5)
- moved R14 137.5 mm to (135.2, 107.4), turned to 180 degrees
- moved TP13 135.9 mm to (58.9, 41.9)
- moved TP24 132.7 mm to (65.0, 41.9)
- moved TP7 132.0 mm to (55.8, 38.8)
- moved TP8 132.0 mm to (55.8, 41.9)
- moved TP10 131.8 mm to (58.9, 32.7)
- moved TP11 131.8 mm to (58.9, 35.8)
- moved TP12 131.8 mm to (58.9, 38.8)
- moved TP15 131.8 mm to (61.9, 32.7)
- moved TP16 131.8 mm to (61.9, 35.8)
- moved TP25 128.7 mm to (68.0, 32.7)
- moved TP26 128.7 mm to (68.0, 35.8)
- moved TP27 128.7 mm to (68.0, 38.8)
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- renumbered JP31 to JP29, JP32 to JP30, JP33 to JP31, JP34 to JP32, JP35 to JP33, JP36 to JP34, JP37 to JP35, JP38 to JP36, JP39 to JP37, R9 to R11, R10 to R12, R11 to R13, R12 to R5, R13 to R6
Connections:
- D3 pad 1: Net-(D3-K) -> +BATT
- Q3 pad 3: Net-(D3-K) -> +BATT
- R5 pad 1: unconnected-(R12-Pad1) -> UC_SDA
- R5 pad 2: unconnected-(R12-Pad2) -> +3V3
- R6 pad 1: unconnected-(R13-Pad1) -> UC_SCL
- R6 pad 2: unconnected-(R13-Pad2) -> +3V3
- R7 pad 2: Net-(JP12-B) -> Net-(JP10-B)
- R8 pad 2: Net-(JP13-B) -> Net-(JP11-B)
- TP10 pad 1: HW_REV_2 -> HW_REV_1
- TP11 pad 1: HW_REV_1 -> HW_REV_2
- TP12 pad 1: Net-(D1-A) -> Net-(U2-PD0)
- TP13 pad 1: HW_REV_3 -> UC_RX
- TP14 pad 1: Net-(JP22-A) -> Net-(D1-A)
- TP15 pad 1: Net-(D2-A) -> UC_TX
- TP16 pad 1: HW_REV_4 -> HW_REV_3
- TP23 pad 1: ADC_ALERT_RDY -> Net-(D2-A)
- TP24 pad 1: Net-(U8-AIN0) -> Net-(U2-PC2)
- TP25 pad 1: HALL_SENS_01_S -> Net-(U2-PC3)
- TP26 pad 1: HALL_SENS_02_S -> Net-(U2-PB2)
- TP27 pad 1: HALL_SENS_03_S -> Net-(U2-PC13)
- TP43 pad 1: FDBK_MOTOR_EN -> EMG_2_UC
- TP45 pad 1: FDBK_MOTOR_1_UC2 -> Net-(U7D-+)
- TP46 pad 1: FDBK_MOTOR_FAULT -> Net-(U6D-+)
- TP53 pad 1: FDBK_MOTOR_2_UC1 -> Net-(U9-AIN0)
- TP54 pad 1: FDBK_MOTOR_2_UC2 -> HALL_SENS_01_S
- TP7 pad 1: Net-(JP17-A) -> UC_SCL
- TP8 pad 1: Net-(JP18-A) -> UC_SDA
- U2 pad 1: unconnected-(U2-VBAT-Pad1) -> +3V3
- U2 pad 10: unconnected-(U2-PC2-Pad10) -> Net-(U2-PC2)
- U2 pad 11: unconnected-(U2-PC3-Pad11) -> Net-(U2-PC3)
- U2 pad 12: unconnected-(U2-VSSA-Pad12) -> Earth
- U2 pad 13: unconnected-(U2-VDDA-Pad13) -> +3V3
- U2 pad 14: unconnected-(U2-PA0-Pad14) -> HW_REV_1
- U2 pad 15: unconnected-(U2-PA1-Pad15) -> HW_REV_2
- U2 pad 16: unconnected-(U2-PA2-Pad16) -> HW_REV_3
- U2 pad 17: unconnected-(U2-PA3-Pad17) -> HW_REV_4
- U2 pad 18: Net-(U2-VSS-Pad18) -> Earth
- U2 pad 19: unconnected-(U2-VDD-Pad19) -> +3V3
- U2 pad 2: unconnected-(U2-PC13-Pad2) -> Net-(U2-PC13)
- U2 pad 20: unconnected-(U2-PA4-Pad20) -> MOTOR_1_FAULT
- U2 pad 21: unconnected-(U2-PA5-Pad21) -> MOTOR_2_FAULT
- U2 pad 22: unconnected-(U2-PA6-Pad22) -> MOTOR_3_FAULT
- U2 pad 23: unconnected-(U2-PA7-Pad23) -> FDBK_MOTOR_FAULT
- U2 pad 24: unconnected-(U2-PC4-Pad24) -> ADC_1_ALERT_RDY
- U2 pad 25: unconnected-(U2-PC5-Pad25) -> ADC_2_ALERT_RDY
- U2 pad 26: unconnected-(U2-PB0-Pad26) -> EMG_1_UC
- U2 pad 27: unconnected-(U2-PB1-Pad27) -> EMG_2_UC
- U2 pad 28: unconnected-(U2-PB2-Pad28) -> Net-(U2-PB2)
- U2 pad 29: unconnected-(U2-PB10-Pad29) -> Net-(U2-PB10)
- U2 pad 3: unconnected-(U2-PC14-Pad3) -> Net-(U2-PC14)
- U2 pad 30: unconnected-(U2-PB11-Pad30) -> Net-(U2-PB11)
- U2 pad 31: Net-(U2-VSS-Pad18) -> Earth
- U2 pad 32: unconnected-(U2-VDD-Pad32) -> +3V3
- U2 pad 33: unconnected-(U2-PB12-Pad33) -> MOTOR_1_EN
- U2 pad 34: unconnected-(U2-PB13-Pad34) -> MOTOR_2_EN
- U2 pad 35: unconnected-(U2-PB14-Pad35) -> MOTOR_3_EN
- U2 pad 36: unconnected-(U2-PB15-Pad36) -> FDBK_MOTOR_EN
- U2 pad 37: unconnected-(U2-PC6-Pad37) -> FDBK_MOTOR_1_UC1
- U2 pad 38: unconnected-(U2-PC7-Pad38) -> FDBK_MOTOR_2_UC1
- U2 pad 39: unconnected-(U2-PC8-Pad39) -> FDBK_MOTOR_1_UC2
- U2 pad 4: unconnected-(U2-PC15-Pad4) -> Net-(U2-PC15)
- U2 pad 40: unconnected-(U2-PC9-Pad40) -> FDBK_MOTOR_2_UC2
- U2 pad 41: unconnected-(U2-PA8-Pad41) -> MOTOR_1_UC1
- U2 pad 42: unconnected-(U2-PA9-Pad42) -> MOTOR_2_UC1
- U2 pad 43: unconnected-(U2-PA10-Pad43) -> MOTOR_3_UC1
- U2 pad 44: unconnected-(U2-PA11-Pad44) -> MOTOR_1_UC2
- U2 pad 45: unconnected-(U2-PA12-Pad45) -> MOTOR_2_UC2
- U2 pad 46: unconnected-(U2-PA13-Pad46) -> JTAG_TMS
- U2 pad 47: Net-(U2-VSS-Pad18) -> Earth
- U2 pad 48: unconnected-(U2-VDD-Pad48) -> +3V3
- U2 pad 49: unconnected-(U2-PA14-Pad49) -> JTAG_TCK
- U2 pad 5: unconnected-(U2-PD0-Pad5) -> Net-(U2-PD0)
- U2 pad 50: unconnected-(U2-PA15-Pad50) -> JTAG_TDI
- U2 pad 51: unconnected-(U2-PC10-Pad51) -> MOTOR_3_UC2
- U2 pad 52: unconnected-(U2-PC11-Pad52) -> LED_1
- U2 pad 53: unconnected-(U2-PC12-Pad53) -> LED_2
- U2 pad 54: unconnected-(U2-PD2-Pad54) -> Net-(U2-PD2)
- U2 pad 55: unconnected-(U2-PB3-Pad55) -> JTAG_TDO
- U2 pad 56: unconnected-(U2-PB4-Pad56) -> JTAG_RST
- U2 pad 57: unconnected-(U2-PB5-Pad57) -> Net-(U2-PB5)
- U2 pad 58: unconnected-(U2-PB6-Pad58) -> UC_TX
- U2 pad 59: unconnected-(U2-PB7-Pad59) -> UC_RX
- U2 pad 6: unconnected-(U2-PD1-Pad6) -> Net-(U2-PD1)
- U2 pad 61: unconnected-(U2-PB8-Pad61) -> UC_SCL
- U2 pad 62: unconnected-(U2-PB9-Pad62) -> UC_SDA
- U2 pad 63: Net-(U2-VSS-Pad18) -> Earth
- U2 pad 64: unconnected-(U2-VDD-Pad64) -> +3V3
- U2 pad 8: unconnected-(U2-PC0-Pad8) -> Net-(U2-PC0)
- U2 pad 9: unconnected-(U2-PC1-Pad9) -> Net-(U2-PC1)
Other:
- board text added: "+"
- board text added: "BATT"
- board text added: "GND RST TDI TDO TCK TMS"
- board text added: "POT"
- board text removed: "+ -"
- board text removed: "BAT"
- board text removed: "POTS"

Commit message: update schm and pcb again
Parts:
- removed the JP9 at (202.3, 219.8)
- removed the JP9 at (192.6, 112.3)
- removed the R49 at (193.8, 52.6)
- removed the R49 at (193.8, 43.8)
- removed the R50 at (165.6, 48.0)
- removed the R50 at (193.8, 55.6)
- removed the TP43 at (58.9, 50.0)
- removed the TP44 at (58.9, 53.0)
- removed the TP49 at (189.7, 56.2)
- added JP38: JMPR_ESP_USB_P, Jumper:SolderJumper-2_P1.3mm_Bridged_RoundedPad1.0x1.5mm, B.Cu at (144.7, 134.6)
- added JP39: JMPR_ESP_USB_N, Jumper:SolderJumper-2_P1.3mm_Bridged_RoundedPad1.0x1.5mm, B.Cu at (144.8, 131.8)
- added JP40: JMPR_ESP_SCL, Jumper:SolderJumper-2_P1.3mm_Bridged_RoundedPad1.0x1.5mm, B.Cu at (121.2, 130.2)
- added JP41: JMPR_ESP_SDA, Jumper:SolderJumper-2_P1.3mm_Bridged_RoundedPad1.0x1.5mm, B.Cu at (121.2, 133.9)
- added JP9: JMPR_TRIM_2, Jumper:SolderJumper-2_P1.3mm_Bridged_RoundedPad1.0x1.5mm, F.Cu at (192.5, 112.3)
- added R49: 18k, Resistor_SMD:R_0805_2012Metric_Pad1.20x1.40mm_HandSolder, F.Cu at (184.7, 79.5)
- added R50: 18k, Resistor_SMD:R_0805_2012Metric_Pad1.20x1.40mm_HandSolder, F.Cu at (184.7, 82.5)
- added TP80: TP_ESP_SCL, TestPoint:TestPoint_Pad_D1.0mm, B.Cu at (134.1, 139.1)
- added TP81: TP_ESP_SDA, TestPoint:TestPoint_Pad_D1.0mm, B.Cu at (131.5, 139.1)
- added U14: ESP32-S3-WROOM-1, Espressif:ESP32-S3-WROOM-1, B.Cu at (132.6, 125.6)
- JP10, JP11, JP12, JP13, JP15, JP16, JP17, JP18, JP29, JP30, JP31, JP32, JP33, JP34, JP35, JP36, JP37, R10, R7, R8, R9: moved to B.Cu
- TP13: renamed from TP16; moved to B.Cu
- TP14: renamed from TP17; moved to B.Cu
- TP15: renamed from TP18; moved to B.Cu
- TP16: renamed from TP19; moved to B.Cu
- TP17: renamed from TP20; moved to B.Cu
- TP18: renamed from TP22; moved to B.Cu
- TP20: renamed from TP24; moved to B.Cu
- TP21: renamed from TP25; moved to B.Cu
- TP22: renamed from TP26; moved to B.Cu
- TP23: renamed from TP27; moved to B.Cu
- TP24: renamed from TP28; moved to B.Cu
- TP25: renamed from TP29; moved to B.Cu
- TP26: renamed from TP30; moved to B.Cu
- TP27: renamed from TP31; moved to B.Cu
- TP28: renamed from TP32; moved to B.Cu
- TP53: renamed from TP57; moved to B.Cu
- TP54: renamed from TP58; moved to B.Cu
- TP59: renamed from TP63; moved to B.Cu
- TP60: renamed from TP64; moved to B.Cu
- TP61: renamed from TP65; moved to B.Cu
- TP62: renamed from TP66; moved to B.Cu
- TP67: renamed from TP71; moved to B.Cu
- TP7: renamed from TP10; moved to B.Cu
- TP72: renamed from TP76; moved to B.Cu
- TP73: renamed from TP77; moved to B.Cu
- TP74: renamed from TP78; moved to B.Cu
- TP75: renamed from TP79; moved to B.Cu
- TP78: renamed from TP82; moved to B.Cu
- TP79: renamed from TP83; moved to B.Cu
- TP8: renamed from TP11; moved to B.Cu
- TP9: renamed from TP12; moved to B.Cu
- moved TP76 185.6 mm to (208.3, 137.0)
- moved TP69 183.1 mm to (202.2, 137.0)
- moved TP77 181.9 mm to (205.8, 137.0)
- moved TP64 179.7 mm to (198.9, 137.0)
- moved TP57 177.1 mm to (192.9, 137.0)
- moved TP66 174.5 mm to (196.5, 137.0)
- moved TP63 173.3 mm to (189.5, 137.0)
- moved TP55 172.6 mm to (183.5, 137.0)
- moved TP65 168.0 mm to (187.1, 137.0)
- moved TP67 161.4 mm to (172.3, 135.2), turned to 180 degrees
- moved TP54 159.6 mm to (172.3, 127.3), turned to 180 degrees
- moved TP5 159.3 mm to (191.8, 121.7)
- moved TP74 157.5 mm to (172.3, 132.8), turned to 180 degrees
- moved TP53 156.8 mm to (172.3, 119.3), turned to 180 degrees
- moved TP68 156.8 mm to (171.8, 131.6)
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- renumbered TP13 to TP10, TP14 to TP11, TP15 to TP12, TP23 to TP19, TP33 to TP29, TP34 to TP30, TP35 to TP31, TP36 to TP32, TP37 to TP33, TP38 to TP34, TP39 to TP35, TP40 to TP36, TP41 to TP37, TP42 to TP38, TP45 to TP41, TP46 to TP42, TP47 to TP43, TP48 to TP44, TP49 to TP45, TP50 to TP46, TP51 to TP47, TP52 to TP48, TP53 to TP49, TP7 to TP5, TP54 to TP50, TP55 to TP51, TP56 to TP52, TP59 to TP55, TP60 to TP56, TP61 to TP57, TP62 to TP58, TP8 to TP6, TP67 to TP63, TP68 to TP64, TP69 to TP65, TP70 to TP66, TP72 to TP68, TP73 to TP69, TP74 to TP70, TP75 to TP71, TP80 to TP76, TP81 to TP77
Connections:
- C3 pad 1: Net-(JP1-A) -> UC_RST
- C4 pad 1: Net-(JP6-A) -> UC_BOOT
- TP1 pad 1: Net-(JP1-A) -> UC_RST
- TP4 pad 1: Net-(JP6-A) -> UC_BOOT
- U5 pad 2: +5V -> +BATT
Other:
- board text added: "EMG SENSOR"
- board text added: "EXTRA UC TEST POINTS TO BE PUT ON BACKSIDE"
- board text added: "locked"
- board text removed: "+"
- board text removed: "+ 1 -"
- board text removed: "+ 2 -"
- board text removed: "+ 3 -"
- board text removed: "-"
- board text removed: "1"
- board text removed: "2"
- board text removed: "BATT"
- board text removed: "BOOT"
- board text removed: "BTN"
- board text removed: "EMG"
- board text removed: "HAPTIC"
- board text removed: "MOTORS"
- board text removed: "POS"
- board text removed: "POT"
- board text removed: "RST"
- board text removed: "USB C"
